File: Hardware/1ST_Schematix/1ST_Schematix.kicad_sch (KiCad schematic)
At the start: 0 parts

Commit message: Créa de soft
Parts:
- added U1: STM32G431RBTx, Package_QFP:LQFP-64_10x10mm_P0.5mm, symbol MCU_ST_STM32G4:STM32G431RBTx
Connections:
- new net: U1.15 (VSS), U1.31 (VSS), U1.47 (VSS), U1.63 (VSS)
Changed lines of the file:
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@@
 	(generator_version "10.0")
 	(paper "A4")
+	(symbol
+		(lib_id "MCU_ST_STM32G4:STM32G431RBTx")
+		(at 134.62 77.47 0)
+		(unit 1)
+		(body_style 1)
+		(exclude_from_sim no)
+		(in_bom yes)
+		(on_board yes)
+		(in_pos_files yes)
+		(dnp no)
+		(fields_autoplaced yes)
+		(property "Reference" "U1"
+			(at 139.3033 125.73 0)
+			(show_name no)
+			(do_not_autoplace no)
+			(effects
+				(font
+					(size 1.27 1.27)
+				)
+				(justify left)
+			)
+		)
+		(property "Value" "STM32G431RBTx"
+			(at 139.3033 128.27 0)
+			(show_name no)
+			(do_not_autoplace no)
+			(effects
+				(font
+					(size 1.27 1.27)
+				)
+				(justify left)
+			)
+		)
+		(property "Footprint" "Package_QFP:LQFP-64_10x10mm_P0.5mm"
+			(at 119.38 123.19 0)
+			(hide yes)
+			(show_name no)
+			(do_not_autoplace no)
+			(effects
+				(font
+					(size 1.27 1.27)
+				)
+				(justify right)
+			)
+		)
+		(property "Datasheet" "https://www.st.com/resource/en/datasheet/stm32g431rb.pdf"
+			(at 134.62 77.47 0)
+			(hide yes)
+			(show_name no)
+			(do_not_autoplace no)
+			(effects
+				(font
+					(size 1.27 1.27)
+				)
+			)
+		)
+		(property "Description" "STMicroelectronics Arm Cortex-M4 MCU, 128KB flash, 32KB RAM, 170 MHz, 1.71-3.6V, 52 GPIO, LQFP64"
+			(at 134.62 77.47 0)
+			(hide yes)
+			(show_name no)
+			(do_not_autoplace no)
+			(effects
+				(font
+					(size 1.27 1.27)
+				)
+			)
+		)
+		(pin "8"
+		)
+		(pin "9"
+		)
+		(pin "14"
+		)
+		(pin "10"
+		)
+		(pin "3"
+		)
+		(pin "13"
+		)
+		(pin "11"
+		)
+		(pin "15"
+		)
+		(pin "22"
+		)
+		(pin "18"
+		)
+		(pin "6"
+		)
+		(pin "4"
+		)
+		(pin "20"
+		)
+		(pin "17"
+		)
+		(pin "1"
+		)
+		(pin "21"
+		)
+		(pin "7"
+		)
+		(pin "19"
+		)
+		(pin "16"
+		)
+		(pin "2"
+		)
+		(pin "5"
+		)
+		(pin "12"
+		)
+		(pin "36"
+		)
+		(pin "38"
+		)
+		(pin "26"
+		)
+		(pin "50"
+		)
+		(pin "33"
+		)
+		(pin "30"
+		)
+		(pin "52"
+		)
+		(pin "34"
+		)
+		(pin "54"
+		)
+		(pin "53"
+		)
+		(pin "48"
+		)
+		(pin "39"
+		)
+		(pin "41"
+		)
+		(pin "32"
+		)
+		(pin "47"
+		)
+		(pin "29"
+		)
+		(pin "42"
+		)
+		(pin "31"
+		)
+		(pin "43"
+		)
+		(pin "49"
+		)
+		(pin "45"
+		)
+		(pin "27"
+		)
+		(pin "28"
+		)
+		(pin "25"
+		)
+		(pin "44"
+		)
+		(pin "46"
+		)
+		(pin "37"
+		)
+		(pin "51"
+		)
+		(pin "35"
+		)
+		(pin "40"
+		)
+		(pin "24"
+		)
+		(pin "23"
+		)
+		(pin "55"
+		)
+		(pin "58"
+		)
+		(pin "62"
+		)
+		(pin "56"
+		)
+		(pin "64"
+		)
+		(pin "59"
+		)
+		(pin "60"
+		)
+		(pin "57"
+		)
+		(pin "63"
+		)
+		(pin "61"
+		)
+		(instances
+			(project "1ST_Schematix"
+				(path "/59c2502d-7c28-4023-9b54-15ec9e15e6d4"
+					(reference "U1")
+					(unit 1)
+				)
+			)
+		)
+	)
 	(sheet_instances
 		(path "/"

Commit message: Datasheet et Schematix
Parts:
- removed U1: STM32G431RBTx, Package_QFP:LQFP-64_10x10mm_P0.5mm, symbol MCU_ST_STM32G4:STM32G431RBTx
Other:
- added sheet Power (Power_Inhibot.kicad_sch)
- added sheet STM32 (CPU_Inhibot.kicad_sch)
Changed lines of the file:
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@@
 	(generator_version "10.0")
 	(paper "A4")
-	(symbol
-		(lib_id "MCU_ST_STM32G4:STM32G431RBTx")
-		(at 134.62 77.47 0)
-		(unit 1)
-		(body_style 1)
+	(sheet
+		(at 186.69 39.37)
+		(size 66.04 49.53)
 		(exclude_from_sim no)
 		(in_bom yes)
 		(on_board yes)
-		(in_pos_files yes)
 		(dnp no)
 		(fields_autoplaced yes)
-		(property "Reference" "U1"
-			(at 139.3033 125.73 0)
+		(stroke
+			(width 0.1524)
+			(type solid)
+		)
+		(fill
+			(color 0 0 0 0)
+		)
+		(property "Sheetname" "STM32"
+			(at 186.69 38.6584 0)
 			(show_name no)
 			(do_not_autoplace no)
@@
 					(size 1.27 1.27)
 				)
-				(justify left)
+				(justify left bottom)
 			)
 		)
-		(property "Value" "STM32G431RBTx"
-			(at 139.3033 128.27 0)
+		(property "Sheetfile" "CPU_Inhibot.kicad_sch"
+			(at 186.69 89.4846 0)
 			(show_name no)
 			(do_not_autoplace no)
@@
 					(size 1.27 1.27)
 				)
-				(justify left)
+				(justify left top)
 			)
 		)
-		(property "Footprint" "Package_QFP:LQFP-64_10x10mm_P0.5mm"
-			(at 119.38 123.19 0)
-			(hide yes)
+		(instances
+			(project "1ST_Schematix"
+				(path "/59c2502d-7c28-4023-9b54-15ec9e15e6d4"
+					(page "2")
+				)
+			)
+		)
+	)
+	(sheet
+		(at 34.29 34.29)
+		(size 52.07 46.99)
+		(exclude_from_sim no)
+		(in_bom yes)
+		(on_board yes)
+		(dnp no)
+		(fields_autoplaced yes)
+		(stroke
+			(width 0.1524)
+			(type solid)
+		)
+		(fill
+			(color 0 0 0 0)
+		)
+		(property "Sheetname" "Power"
+			(at 34.29 33.5784 0)
 			(show_name no)
 			(do_not_autoplace no)
@@
 					(size 1.27 1.27)
 				)
-				(justify right)
+				(justify left bottom)
 			)
 		)
-		(property "Datasheet" "https://www.st.com/resource/en/datasheet/stm32g431rb.pdf"
-			(at 134.62 77.47 0)
-			(hide yes)
+		(property "Sheetfile" "Power_Inhibot.kicad_sch"
+			(at 34.29 81.8646 0)
 			(show_name no)
 			(do_not_autoplace no)
@@
 					(size 1.27 1.27)
 				)
+				(justify left top)
 			)
-		)
-		(property "Description" "STMicroelectronics Arm Cortex-M4 MCU, 128KB flash, 32KB RAM, 170 MHz, 1.71-3.6V, 52 GPIO, LQFP64"
-			(at 134.62 77.47 0)
-			(hide yes)
-			(show_name no)
-			(do_not_autoplace no)
-			(effects
-				(font
-					(size 1.27 1.27)
-				)
-			)
-		)
-		(pin "8"
-		)
-		(pin "9"
-		)
-		(pin "14"
-		)
-		(pin "10"
-		)
-		(pin "3"
-		)
-		(pin "13"
-		)
-		(pin "11"
-		)
-		(pin "15"
-		)
-		(pin "22"
-		)
-		(pin "18"
-		)
-		(pin "6"
-		)
-		(pin "4"
-		)
-		(pin "20"
-		)
-		(pin "17"
-		)
-		(pin "1"
-		)
-		(pin "21"
-		)
-		(pin "7"
-		)
-		(pin "19"
-		)
-		(pin "16"
-		)
-		(pin "2"
-		)
-		(pin "5"
-		)
-		(pin "12"
-		)
-		(pin "36"
-		)
-		(pin "38"
-		)
-		(pin "26"
-		)
-		(pin "50"
-		)
-		(pin "33"
-		)
-		(pin "30"
-		)
-		(pin "52"
-		)
-		(pin "34"
-		)
-		(pin "54"
-		)
-		(pin "53"
-		)
-		(pin "48"
-		)
-		(pin "39"
-		)
-		(pin "41"
-		)
-		(pin "32"
-		)
-		(pin "47"
-		)
-		(pin "29"
-		)
-		(pin "42"
-		)
-		(pin "31"
-		)
-		(pin "43"
-		)
-		(pin "49"
-		)
-		(pin "45"
-		)
-		(pin "27"
-		)
-		(pin "28"
-		)
-		(pin "25"
-		)
-		(pin "44"
-		)
-		(pin "46"
-		)
-		(pin "37"
-		)
-		(pin "51"
-		)
-		(pin "35"
-		)
-		(pin "40"
-		)
-		(pin "24"
-		)
-		(pin "23"
-		)
-		(pin "55"
-		)
-		(pin "58"
-		)
-		(pin "62"
-		)
-		(pin "56"
-		)
-		(pin "64"
-		)
-		(pin "59"
-		)
-		(pin "60"
-		)
-		(pin "57"
-		)
-		(pin "63"
-		)
-		(pin "61"
 		)
 		(instances
 			(project "1ST_Schematix"
 				(path "/59c2502d-7c28-4023-9b54-15ec9e15e6d4"
-					(reference "U1")
-					(unit 1)
+					(page "3")
 				)
 			)

Commit message: PCB
Other:
- added sheet Sensor (Sensor_Inhibot.kicad_sch)
Changed lines of the file:
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@@
+		)
+	)
+	(sheet
+		(at 95.25 97.79)
+		(size 74.93 50.8)
+		(exclude_from_sim no)
+		(in_bom yes)
+		(on_board yes)
+		(dnp no)
+		(fields_autoplaced yes)
+		(stroke
+			(width 0.1524)
+			(type solid)
+		)
+		(fill
+			(color 0 0 0 0)
+		)
+		(property "Sheetname" "Sensor"
+			(at 95.25 97.0784 0)
+			(show_name no)
+			(do_not_autoplace no)
+			(effects
+				(font
+					(size 1.27 1.27)
+				)
+				(justify left bottom)
+			)
+		)
+		(property "Sheetfile" "Sensor_Inhibot.kicad_sch"
+			(at 95.25 149.1746 0)
+			(show_name no)
+			(do_not_autoplace no)
+			(effects
+				(font
+					(size 1.27 1.27)
+				)
+				(justify left top)
+			)
+		)
+		(instances
+			(project "1ST_Schematix"
+				(path "/59c2502d-7c28-4023-9b54-15ec9e15e6d4"
+					(page "4")
+				)
+			)
 		)
 	)

Commit message: Update KiCad + Création Soft_Inhibot.ioc
Soft_Inhibot est mieux que juste Software. C'est mon avis...
Parts:
- added H1, H2, H3, H4: MountingHole_Pad, MountingHole:MountingHole_3.2mm_M3_ISO14580_Pad, symbol Mechanical:MountingHole_Pad
Connections:
- new net GND: H1.1, H2.1, H3.1, H4.1
Other:
- added sheet Connectors (Connector_Inhibot.kicad_sch)
- sheet Power ports: added BMS_SCL, BMS_SDA, BMS_~{INT}, STM32_D+, STM32_D-, VBAT, ~{QON}; removed none
- sheet STM32 ports: added D+, D-, ENCODER1_CH1, ENCODER1_CH2, ENCODER2_CH1, ENCODER2_CH2, INTERRUPT3, QON, SCL, SCL1, SDA, SDA1, TIM1_RGB, TIM2_PWM_DRIVER1, TIM2_PWM_DRIVER2, TIM2_PWM_DRIVER3, TIM2_PWM_DRIVER4, TIM2_PWM_SERVO, Uart4_RX, Uart4_TX; removed none
- sheet Sensor ports: added AOUT1, AOUT2, BOUT1, BOUT2, INT1_Mag, INT2_Mag, PWM1, PWM2, PWM3, PWM4, SCL_Mag, SDA_Mag, VM; removed none
- title: (none) -> Inhibot

Commit message: Update PCB
Parts:
- added R17: 10k, Resistor_SMD:R_0402_1005Metric_Pad0.72x0.64mm_HandSolder, symbol Device:R
- added SW1: SW_Push, Button_Switch_SMD:SW_Push_1P1T_NO_CK_KMR2, symbol Switch:SW_Push
Connections:
- net GND: now also SW1.1
- net Power/~{QON}: now also R17.2, SW1.2
- new net +3.3V: R17.1
Other:
- sheet Connectors ports: added INT1_Mag, INT2_Mag, INT_Color, RX_Bluetooth, SCL_Color, SCL_Mag_conn, SCL_TOF, SDA_Color, SDA_Mag_conn, SDA_TOF, TOF1_GPIO1, TOF1_XST, TOF2_GPIO1, TOF2_XST, TX_Bluetooth; removed none
- sheet STM32 ports: added none; removed SCL, SDA
- note added: "Button ON/OFF"

Commit message: ehe
Changed lines of the file:
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@@
 		(color 0 0 0 0)
+	)
+	(bus_entry
+		(at 36.83 8.89)
+		(size 2.54 2.54)
+		(stroke
+			(width 0)
+			(type default)
+		)
+	)
+	(bus_entry
+		(at 44.45 39.37)
+		(size 2.54 2.54)
+		(stroke
+			(width 0)
+			(type default)
+		)
 	)
 	(wire

Commit message: nom des compo
Parts:
- renumbered H1 to H101, H2 to H102, H3 to H103, H4 to H104, R17 to R101, SW1 to SW101
Changed lines of the file:
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@@
 		(dnp no)
 		(fields_autoplaced yes)
-		(property "Reference" "SW1"
+		(property "Reference" "SW101"
 			(at 86.36 82.5499 90)
 			(show_name no)
@@
 			(project "1ST_Schematix"
 				(path "/59c2502d-7c28-4023-9b54-15ec9e15e6d4"
-					(reference "SW1")
+					(reference "SW101")
 					(unit 1)
 				)
@@
 		(dnp no)
 		(fields_autoplaced yes)
-		(property "Reference" "H3"
+		(property "Reference" "H103"
 			(at 254 135.8899 0)
 			(show_name no)
@@
 			(project "1ST_Schematix"
 				(path "/59c2502d-7c28-4023-9b54-15ec9e15e6d4"
-					(reference "H3")
+					(reference "H103")
 					(unit 1)
 				)
@@
 		(dnp no)
 		(fields_autoplaced yes)
-		(property "Reference" "H4"
+		(property "Reference" "H104"
 			(at 261.62 135.8899 0)
 			(show_name no)
@@
 			(project "1ST_Schematix"
 				(path "/59c2502d-7c28-4023-9b54-15ec9e15e6d4"
-					(reference "H4")
+					(reference "H104")
 					(unit 1)
 				)
@@
 		(dnp no)
 		(fields_autoplaced yes)
-		(property "Reference" "#PWR040"
+		(property "Reference" "#PWR0101"
 			(at 85.09 63.5 0)
 			(hide yes)
@@
 			(project "1ST_Schematix"
 				(path "/59c2502d-7c28-4023-9b54-15ec9e15e6d4"
-					(reference "#PWR040")
+					(reference "#PWR0101")
 					(unit 1)
 				)
@@
 		(dnp no)
 		(fields_autoplaced yes)
-		(property "Reference" "#PWR023"
+		(property "Reference" "#PWR0103"
 			(at 247.65 149.86 0)
 			(hide yes)
@@
 			(project "1ST_Schematix"
 				(path "/59c2502d-7c28-4023-9b54-15ec9e15e6d4"
-					(reference "#PWR023")
+					(reference "#PWR0103")
 					(unit 1)
 				)
@@
 		(dnp no)
 		(fields_autoplaced yes)
-		(property "Reference" "H1"
+		(property "Reference" "H101"
 			(at 238.76 135.8899 0)
 			(show_name no)
@@
 			(project "1ST_Schematix"
 				(path "/59c2502d-7c28-4023-9b54-15ec9e15e6d4"
-					(reference "H1")
+					(reference "H101")
 					(unit 1)
 				)
@@
 		(dnp no)
 		(fields_autoplaced yes)
-		(property "Reference" "H2"
+		(property "Reference" "H102"
 			(at 246.38 135.8899 0)
 			(show_name no)
@@
 			(project "1ST_Schematix"
 				(path "/59c2502d-7c28-4023-9b54-15ec9e15e6d4"
-					(reference "H2")
+					(reference "H102")
 					(unit 1)
 				)
@@
 		(in_pos_files yes)
 		(dnp no)
-		(property "Reference" "R17"
+		(property "Reference" "R101"
 			(at 89.916 65.278 0)
 			(show_name no)
@@
 			(project "1ST_Schematix"
 				(path "/59c2502d-7c28-4023-9b54-15ec9e15e6d4"
-					(reference "R17")
+					(reference "R101")
 					(unit 1)
 				)
@@
 		(dnp no)
 		(fields_autoplaced yes)
-		(property "Reference" "#PWR041"
+		(property "Reference" "#PWR0102"
 			(at 85.09 96.52 0)
 			(hide yes)
@@
 			(project "1ST_Schematix"
 				(path "/59c2502d-7c28-4023-9b54-15ec9e15e6d4"
-					(reference "#PWR041")
-					(unit 1)
-				)
+					(reference "#PWR0102")
+					(unit 1)
+				)

Commit message: Update
Parts:
- R101: now not fitted
Other:
- sheet Power ports: added Jauge_SCL, Jauge_SDA; removed none
- sheet STM32 ports: added SCL2, SDA2; removed none
