File: Hardware/1ST_Schematix/_autosave-Power_Inhibot.kicad_sch (KiCad schematic)
At the start: 2 parts, among them J1 USB_C_Receptacle_PowerOnly_24P, U2 BQ25895RTW

Commit message: Kicad
Parts:
- added U3: LP2985-3.3, Package_TO_SOT_SMD:SOT-23-5, symbol Regulator_Linear:LP2985-3.3
Connections:
- net GND: now reaches J1.A1 (GND), J1.A12 (GND), J1.B1 (GND), J1.B12 (GND)
- net at J1.A4 (VBUS), J1.A9 (VBUS), J1.B4 (VBUS)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: now also U2.1 (VBUS)
- no-connect marks 0 -> 2
Other:
- moved on the sheet: J1, U2
