File: Hardware/1ST_Schematix/CPU_Inhibot.kicad_sch (KiCad schematic)
At the start: 1 part, among them U1 STM32G431RBTx

Commit message: stm pinout
Parts:
- added C101: 4u7, Capacitor_SMD:C_0603_1608Metric, symbol Device:C_Small
- added C102, C103, C114: 100n, Capacitor_SMD:C_0402_1005Metric, symbol Device:C_Small
- added C106: 10n, Capacitor_SMD:C_0402_1005Metric, symbol Device:C_Small
- added SW102: SW_Push, Button_Switch_SMD:SW_SPST_B3U-3000P, symbol Switch:SW_Push
Connections:
- net TIM2_PWM1: now reaches U1.12 (PA0)
- net TIM2_PWM2: now reaches U1.13 (PA1)
- net TIM2_PWM3: now reaches U1.14 (PA2)
- net GND: now reaches U1.15 (VSS), U1.31 (VSS), U1.47 (VSS), U1.63 (VSS)
- net GND: now also U1.27 (VSSA), C101.2, C102.2, C103.2, C106.2, C114.2, SW102.2
- net +3.3V: now reaches U1.16 (VDD)
- net +3.3V: now also U1.29 (VDDA), U1.32 (VDD), U1.48 (VDD), U1.64 (VDD), C101.1, C102.1, C103.1, C106.1
- net TIM2_PWM4: now reaches U1.17 (PA3)
- net SCL: now reaches U1.49 (PA13)
- net SDA: now reaches U1.50 (PA14)
- net Uart4_TX: now reaches U1.52 (PC10)
- net Uart4_RX: now reaches U1.53 (PC11)
- net NRST: now reaches U1.7 (PG10)
- net NRST: now also C114.1, SW102.1

Commit message: modification ioc et UC
Parts:
- added C104, C105: 10pF, Capacitor_SMD:C_0603_1608Metric, symbol Device:C_Small
- added D1: LED_Small, LED_SMD:LED_Cree-XHP50_3V_HighDensity, symbol Device:LED_Small
- added D2: LED_Small, symbol Device:LED_Small
- added J102: Conn_ST_STDC14, Connector_PinHeader_1.27mm:PinHeader_2x07_P1.27mm_Vertical_SMD, symbol Connector:Conn_ST_STDC14
- added R1, R2, R3: R_Small, Resistor_THT:R_Array_SIP4, symbol Device:R_Small
- added Y1: Crystal_GND24_Small, Package_DFN_QFN:WDFN-10-1EP_3x3mm_P0.5mm_EP1.8x2.5mm, symbol Device:Crystal_GND24_Small
Connections:
- net +3.3V: now also D1.2 (A), J102.3 (VCC)
- net GND: now also C104.1, C105.1, J102.11 (GNDDetect), J102.5 (GND), J102.7 (GND), R2.1, R3.1, Y1.2 (G), Y1.4 (G)
- net NRST: now also J102.12 (~{RST})
- net SCL: now also U1.51 (PA15); no longer U1.49 (PA13)
- net SDA: now also U1.62 (PB9); no longer U1.50 (PA14)
- net TIM2_PWM_SERVO: now reaches U1.20 (PA6)
- net TIM2_PWM_DRIVER3: now reaches U1.30 (PB10)
- net TIM2_PWM_DRIVER4: now reaches U1.33 (PB11)
- net SYS_SWDIO: now reaches U1.35 (PB13)
- net SYS_SWDIO: now also J102.4 (JTMS/SWDIO)
- net SYS_SWCLK: now reaches U1.36 (PB14)
- net SYS_SWCLK: now also J102.6 (JCLK/SWCLK)
- net D-: now reaches U1.45 (PA11)
- net D+: now reaches U1.46 (PA12)
- net RCC_OSC_IN: now reaches U1.5 (PF0)
- net RCC_OSC_IN: now also C105.2, Y1.1
- net ENCODER1_CH1: now reaches U1.59 (PB6)
- net at U1.6 (PF1): now also R1.2
- net ENCODER1_CH2: now reaches U1.60 (PB7)
- net QON: now reaches U1.8 (PC0)
- net TIM2_PWM1 renamed TIM2_PWM_DRIVER1
- net TIM2_PWM2 renamed TIM2_PWM_DRIVER2
- net TIM2_PWM3 renamed USART2_TX
- net USART2_TX: now also J102.14 (VCP_TX)
- net TIM2_PWM4 renamed USART2_RX
- net USART2_RX: now also J102.13 (VCP_RX)
- new net: D1.1 (K), R2.2
- new net: C104.2, R1.1, Y1.3
- new net: D2.1 (K), R3.2
- new net LED_STATUS: D2.2 (A)
- no-connect marks 0 -> 3
Other:
- note added: "Misc"
- note added: "Programmer"
- note added: "STM"

Commit message: more modif
Parts:
- added R4: 100k, Resistor_THT:R_Array_SIP4, symbol Device:R_Small
- D1: value LED_Small -> GREEN
- D2: value LED_Small -> RED
- R2, R3: value R_Small -> 1k
Connections:
- net GND: now also R4.1
- net RCC_OSC_OUT: now also R1.2, U1.6 (PF1)
- net INTERRUPT3: now reaches U1.11 (PC3)
- net BOOT0: now reaches U1.42 (PA8)
- net BOOT0: now also R4.2

Commit message: Update KiCad + Création Soft_Inhibot.ioc
Soft_Inhibot est mieux que juste Software. C'est mon avis...
Parts:
- added JP1, JP2: SolderJumper_2_Open, Jumper:SolderJumper-2_P1.3mm_Open_TrianglePad1.0x1.5mm, symbol Jumper:SolderJumper_2_Open
- added R15, R16: 4.7k, Resistor_THT:R_Array_SIP4, symbol Device:R_Small
Connections:
- net +3.3V: now also R15.2, R16.2
- net ENCODER1_CH1: now also U1.38 (PC6)
- net ENCODER1_CH2: now also U1.39 (PC7)
- net QON: now also U1.24 (PB0); no longer U1.8 (PC0)
- net USART2_RX: now also JP1.2 (B); no longer J102.13 (VCP_RX)
- net USART2_TX: now also JP2.2 (B); no longer J102.14 (VCP_TX)
- net SCL renamed SCL1
- net SCL1: now also R15.1
- net SDA renamed SDA1
- net SDA1: now also R16.1
- new net: J102.14 (VCP_TX), JP2.1 (A)
- new net: J102.13 (VCP_RX), JP1.1 (A)
- new net TIM1_RGB: U1.8 (PC0)
Other:
- note added: "STM32"
- note removed: "STM"
- title: (none) -> Inhibot

Commit message: Update PCB
Connections:
- net ENCODER1_CH1: no longer U1.59 (PB6)
- net ENCODER1_CH2: no longer U1.60 (PB7)
- new net ENCODER2_CH1: U1.59 (PB6)
- new net ENCODER2_CH2: U1.60 (PB7)
Changed lines of the file:
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@@
 		)
 	)
-	(hierarchical_label "ENCODER1_CH2"
+	(hierarchical_label "ENCODER2_CH2"
 		(shape output)
 		(at 115.57 105.41 0)
@@
 	)
 	(hierarchical_label "SCL1"
-		(shape input)
+		(shape bidirectional)
 		(at 203.2 100.33 0)
 		(effects
@@
 	)
 	(hierarchical_label "Uart4_TX"
-		(shape input)
+		(shape output)
 		(at 74.93 92.71 180)
 		(effects
@@
 		)
 	)
-	(hierarchical_label "ENCODER1_CH1"
+	(hierarchical_label "ENCODER2_CH1"
 		(shape output)
 		(at 115.57 102.87 0)
@@
 	)
 	(hierarchical_label "SDA1"
-		(shape input)
+		(shape bidirectional)
 		(at 203.2 104.14 0)
 		(effects
@@
 	)
 	(hierarchical_label "Uart4_RX"
-		(shape input)
+		(shape output)
 		(at 74.93 95.25 180)
 		(effects

Commit message: ehe
Connections:
- net BOOT0: now also U1.61 (PB8); no longer U1.42 (PA8)
Changed lines of the file:
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@@
+	(wire
+		(pts
+			(xy 114.3 107.95) (xy 120.65 107.95)
+		)
+		(stroke
+			(width 0)
+			(type default)
+		)
+	)
 	(wire
 		(pts
@@
 		(pts
 			(xy 74.93 92.71) (xy 78.74 92.71)
-		)
-		(stroke
-			(width 0)
-			(type default)
-		)
-	)
-	(wire
-		(pts
-			(xy 114.3 64.77) (xy 120.65 64.77)
 		)
 		(stroke
@@
 		)
 	)
-	(label "BOOT0"
-		(at 120.65 64.77 0)
-		(effects
-			(font
-				(size 1.27 1.27)
-			)
-			(justify left bottom)
-		)
-	)
 	(label "NRST"
 		(at 69.85 49.53 180)
@@
 		)
 	)
+	(label "BOOT0"
+		(at 120.65 107.95 0)
+		(effects
+			(font
+				(size 1.27 1.27)
+			)
+			(justify left bottom)
+		)
+	)
