File: Hardware/1ST_Schematix/CPU_Inhibot.kicad_sch (KiCad schematic)
At the start: 22 parts, among them J201 Conn_ST_STDC14, SW201 SW_Push, U201 STM32G431RBTx, Y201 X322516MLB4SI

Commit message: routage à faire vérifier
Connections:
- net TIM2_PWM_SERVO renamed TIM2_PWM_SERVO1
- net TIM2_PWM_SERVO1: no longer U201.21 (PA7)
- new net TIM2_PWM_SERVO2: U201.21 (PA7)
Changed lines of the file:
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@@
 		)
 	)
-	(hierarchical_label "TIM2_PWM_SERVO"
+	(hierarchical_label "TIM2_PWM_SERVO2"
 		(shape output)
 		(at 116.84 62.23 0)
@@
 		)
 	)
-	(hierarchical_label "TIM2_PWM_SERVO"
+	(hierarchical_label "TIM2_PWM_SERVO1"
 		(shape output)
 		(at 116.84 59.69 0)
