File: Hardware/1ST_Schematix/Power_Inhibot.kicad_sch (KiCad schematic)
At the start: 2 parts, among them J1 USB_C_Receptacle_PowerOnly_24P, U2 BQ25895RTW

Commit message: Power
Parts:
- added C1, C2, C3, C4, C5: C, symbol Device:C
- added L1: L, Package_SO:SOIC-16_3.9x9.9mm_P1.27mm, symbol Device:L
- added R1, R2, R3, R4, R5: R, symbol Device:R
- added U3: LP2985-3.3, Package_TO_SOT_SMD:SOT-23-5, symbol Regulator_Linear:LP2985-3.3
Connections:
- net GND: now reaches J1.A1 (GND), J1.A12 (GND), J1.B1 (GND), J1.B12 (GND)
- net GND: now also J1.SH (SHIELD), U2.17 (PGND), U2.18 (PGND), U2.25 (PGND), C1.2, C2.2, C3.2, C5.1, R1.2, R2.2, R4.2, R5.1
- net at J1.A4 (VBUS), J1.A9 (VBUS), J1.B4 (VBUS)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: now also U2.1 (VBUS), C1.1
- net at J1.A5 (CC1): now also R1.1
- net at J1.B5 (CC2): now also R2.1
- net at U2.10 (ILIM): now also R5.2
- net at U2.11 (TS): now also R3.2, R4.1
- net VBAT: now reaches U2.13 (BAT), U2.14 (BAT)
- net VBAT: now also C2.1, C3.1
- net SYS: now reaches U2.15 (SYS), U2.16 (SYS)
- net SYS: now also L1.2, U3.1 (VIN)
- net at U2.19 (SW), U2.20 (SW): now also C4.2, L1.1
- net at U2.21 (BTST): now also C4.1
- net at U2.22 (REGN): now also C5.2, R3.1
- net BMS_SCL: now reaches U2.5 (SCL)
- net BMS_SDA: now reaches U2.6 (SDA)
Other:
- moved on the sheet: J1, U2

Commit message: PCB
Parts:
- removed J1: USB_C_Receptacle_PowerOnly_24P, Package_DFN_QFN:WDFN-10-1EP_3x3mm_P0.5mm_EP1.8x2.5mm, symbol Connector:USB_C_Receptacle_PowerOnly_24P
- removed U2: BQ25895RTW, Package_DFN_QFN:Texas_RTW_WQFN-24-1EP_4x4mm_P0.5mm_EP2.7x2.7mm, symbol Battery_Management:BQ25895RTW
- added J1: USB_C_Receptacle_USB2.0_16P, Connector_USB:USB_C_Receptacle_GCT_USB4105-xx-A_16P_TopMnt_Horizontal, symbol Connector:USB_C_Receptacle_USB2.0_16P
- added U2: BQ25896RTW, Package_DFN_QFN:Texas_RTW_WQFN-24-1EP_4x4mm_P0.5mm_EP2.7x2.7mm, symbol inhibot_lib:BQ25896RTW
Connections:
- net BMS_SCL: now also U2.5 (SCL)
- net BMS_SDA: now also U2.6 (SDA)
- net GND: now also J1.A1 (GND), J1.A12 (GND), J1.B1 (GND), J1.B12 (GND), J1.SH (SHIELD), U2.17 (PGND), U2.18 (PGND), U2.25 (PGND)
- net SYS: now also U2.15 (SYS), U2.16 (SYS)
- net VBAT: now also U2.13 (BAT), U2.14 (BAT)
- net at C1.1: now also U2.1 (VBUS)
- net at C4.1: now also U2.21 (BTST)
- net at C4.2, L1.1: now also U2.19 (SW), U2.20 (SW)
- net at C5.2, R3.1: now also U2.22 (REGN)
- net at R3.2, R4.1: now also U2.11 (TS)
- net at R5.2: now also U2.10 (ILIM)
- new net: J1.A4 (VBUS), J1.A9 (VBUS), J1.B4 (VBUS), J1.B9 (VBUS)
Other:
- moved on the sheet: R1, R2

Commit message: PCB POWER
Parts:
- removed R1, R2: R, symbol Device:R
- added C10, C11, C6, C7, C8, C9: C, symbol Device:C
- added D1: ~{PG}, Package_DFN_QFN:Texas_RTW_WQFN-24-1EP_4x4mm_P0.5mm_EP2.7x2.7mm_ThermalVias, symbol Device:LED
- added D2: STAT, Package_DFN_QFN:Texas_RTW_WQFN-24-1EP_4x4mm_P0.5mm_EP2.7x2.7mm_ThermalVias, symbol Device:LED
- added R1, R2, R6, R7: 5k1, Resistor_SMD:R_0402_1005Metric, symbol Device:R_Small
- added U4: USBLC6-2SC6, Package_TO_SOT_SMD:SOT-23-6, symbol Power_Protection:USBLC6-2SC6
- C4: value C -> 47u
- C5: value C -> 4.7u
- R3, R4: value R -> 10k
Connections:
- net SYS is gone; now on net +5V: L1.2, U2.15 (SYS), U2.16 (SYS), U3.1 (VIN)
- net GND: now also U2.2 (PSEL), U2.9 (~{CE}), U3.2 (GND), C10.2, C11.2, C6.2, C7.2, C8.2, C9.2, R1.2, R2.2, U4.2 (GND)
- net at J1.A4 (VBUS), J1.A9 (VBUS), J1.B4 (VBUS)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: now also C1.1, U2.1 (VBUS), U4.5 (VBUS)
- net CC1: now reaches J1.A5 (CC1)
- net CC1: now also R2.1
- net USB_D+: now reaches J1.A6 (D+)
- net USB_D+: now also J1.B6 (D+), U4.3 (I/O2)
- net USB_D-: now reaches J1.A7 (D-)
- net USB_D-: now also J1.B7 (D-), U4.1 (I/O1)
- net CC2: now reaches J1.B5 (CC2)
- net CC2: now also R1.1
- net ~{QON}: now reaches U2.12 (~{QON})
- net at U2.23 (PMID): now also C6.1
- net ~{PG}: now reaches U2.3 (~{PG})
- net ~{PG}: now also R6.2
- net STAT: now reaches U2.4 (STAT)
- net STAT: now also R7.2
- net ~{INT}: now reaches U2.7 (~{INT})
- net OTG: now reaches U2.8 (OTG)
- net +5V: now reaches U3.3 (ON/~{OFF})
- net +5V: now also C10.1, C11.1, C7.1, D1.2 (A), D2.2 (A)
- net at U3.4 (BP): now also C9.1
- net +3.3V: now reaches U3.5 (VOUT)
- net +3.3V: now also C8.1
- new net: D2.1 (K), R7.1
- new net: D1.1 (K), R6.1
- new net STM32_D+: U4.4 (I/O2)
- new net STM32_D-: U4.6 (I/O1)
- no-connect marks 0 -> 3
Other:
- moved on the sheet: C1, C2, C3, C4, C5, J1, L1, R3, R4, R5, U2, U3

Commit message: Update Power
Parts:
- added R11, R12: 1k, symbol Device:R
Connections:
- net GND: now also R11.2, R12.2; no longer U2.2 (PSEL)
- net OTG: no longer names the net of U2.8 (OTG)
- net OTG: now also R11.1
- net ~{INT} renamed BMS_~{INT}
- new net: R12.1, U2.2 (PSEL)
Changed lines of the file:
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@@
 	)
 	(junction
+		(at 113.03 91.44)
+		(diameter 0)
+		(color 0 0 0 0)
+	)
+	(junction
 		(at 184.15 101.6)
 		(diameter 0)
@@
 	(wire
 		(pts
+			(xy 113.03 91.44) (xy 113.03 95.25)
+		)
+		(stroke
+			(width 0)
+			(type default)
+		)
+	)
+	(wire
+		(pts
 			(xy 27.94 113.03) (xy 27.94 115.57)
 		)
@@
 	(wire
 		(pts
+			(xy 118.11 73.66) (xy 113.03 73.66)
+		)
+		(stroke
+			(width 0)
+			(type default)
+		)
+	)
+	(wire
+		(pts
 			(xy 156.21 104.14) (xy 156.21 106.68)
 		)
@@
 	(wire
 		(pts
+			(xy 113.03 91.44) (xy 118.11 91.44)
+		)
+		(stroke
+			(width 0)
+			(type default)
+		)
+	)
+	(wire
+		(pts
 			(xy 31.75 106.68) (xy 31.75 113.03)
 		)
@@
 	(wire
 		(pts
-			(xy 135.89 73.66) (xy 115.57 73.66)
+			(xy 135.89 73.66) (xy 125.73 73.66)
 		)
 		(stroke
@@
 	(wire
 		(pts
+			(xy 125.73 91.44) (xy 135.89 91.44)
+		)
+		(stroke
+			(width 0)
+			(type default)
+		)
+	)
+	(wire
+		(pts
 			(xy 170.18 118.11) (xy 170.18 116.84)
 		)
@@
 	(wire
 		(pts
-			(xy 115.57 73.66) (xy 115.57 74.93)
+			(xy 113.03 73.66) (xy 113.03 91.44)
 		)
 		(stroke
@@
 		)
 	)
-	(hierarchical_label "OTG"
-		(shape bidirectional)
-		(at 135.89 91.44 180)
-		(effects
-			(font
-				(size 1.27 1.27)
-			)
-			(justify right)
-		)
-	)
 	(hierarchical_label "STM32_D-"
 		(shape bidirectional)
@@
 		)
 	)
-	(hierarchical_label "~{INT}"
+	(hierarchical_label "BMS_~{INT}"
 		(shape bidirectional)
 		(at 135.89 88.9 180)
@@
 	(symbol
 		(lib_id "power:GND")
-		(at 115.57 74.93 0)
+		(at 113.03 95.25 0)
 		(unit 1)
 		(body_style 1)
@@
 		(fields_autoplaced yes)
 		(property "Reference" "#PWR06"
-			(at 115.57 81.28 0)
+			(at 113.03 101.6 0)
 			(hide yes)
 			(show_name no)
@@
 		)
 		(property "Value" "GND"
-			(at 115.57 80.01 0)
+			(at 113.03 100.33 0)
 			(show_name no)
 			(do_not_autoplace no)
@@
 		)
 		(property "Footprint" "Package_TO_SOT_SMD:SOT-23-5"
-			(at 115.57 74.93 0)
+			(at 113.03 95.25 0)
 			(hide yes)
 			(show_name no)
@@
 		)
 		(property "Datasheet" ""
-			(at 115.57 74.93 0)
+			(at 113.03 95.25 0)
 			(hide yes)
 			(show_name no)
@@
 		)
 		(property "Description" "Power symbol creates a global label with name \"GND\" , ground"
-			(at 115.57 74.93 0)
+			(at 113.03 95.25 0)
 			(hide yes)
 			(show_name no)
@@
 	)
 	(symbol
+		(lib_id "Device:R")
+		(at 121.92 73.66 270)
+		(unit 1)
+		(body_style 1)
+		(exclude_from_sim no)
+		(in_bom yes)
+		(on_board yes)
+		(in_pos_files yes)
+		(dnp no)
+		(fields_autoplaced yes)
+		(property "Reference" "R12"
+			(at 121.92 67.31 90)
+			(show_name no)
+			(do_not_autoplace no)
+			(effects
+				(font
+					(size 1.27 1.27)
+				)
+			)
+		)
+		(property "Value" "1k"
+			(at 121.92 69.85 90)
+			(show_name no)
+			(do_not_autoplace no)
+			(effects
+				(font
+					(size 1.27 1.27)
+				)
+			)
+		)
+		(property "Footprint" ""
+			(at 121.92 71.882 90)
+			(hide yes)
+			(show_name no)
+			(do_not_autoplace no)
+			(effects
+				(font
+					(size 1.27 1.27)
+				)
+			)
+		)
+		(property "Datasheet" ""
+			(at 121.92 73.66 0)
+			(hide yes)
+			(show_name no)
+			(do_not_autoplace no)
+			(effects
+				(font
+					(size 1.27 1.27)
+				)
+			)
+		)
+		(property "Description" "Resistor"
+			(at 121.92 73.66 0)
+			(hide yes)
+			(show_name no)
+			(do_not_autoplace no)
+			(effects
+				(font
+					(size 1.27 1.27)
+				)
+			)
+		)
+		(pin "2"
+		)
+		(pin "1"
+		)
+		(instances
+			(project "1ST_Schematix"
+				(path "/59c2502d-7c28-4023-9b54-15ec9e15e6d4/58991d82-9dd2-4511-b974-9bfcbd0b4f51"
+					(reference "R12")
+					(unit 1)
+				)
+			)
+		)
+	)
+	(symbol
 		(lib_id "Device:C")
 		(at 162.56 82.55 180)
@@
 					(unit 1)
 				)
+			)
+		)
+	)
+	(symbol
+		(lib_id "Device:R")
+		(at 121.92 91.44 270)
+		(unit 1)
+		(body_style 1)
+		(exclude_from_sim no)
+		(in_bom yes)
+		(on_board yes)
+		(in_pos_files yes)
+		(dnp no)
+		(fields_autoplaced yes)
+		(property "Reference" "R11"
+			(at 121.92 85.09 90)
+			(show_name no)
+			(do_not_autoplace no)
+			(effects
+				(font
+					(size 1.27 1.27)
+				)
+			)
+		)
+		(property "Value" "1k"
+			(at 121.92 87.63 90)
+			(show_name no)
+			(do_not_autoplace no)
+			(effects
+				(font
+					(size 1.27 1.27)
+				)
+			)
+		)
+		(property "Footprint" ""
+			(at 121.92 89.662 90)
+			(hide yes)
+			(show_name no)
+			(do_not_autoplace no)
+			(effects
+				(font
+					(size 1.27 1.27)
+				)
+			)
+		)
+		(property "Datasheet" ""
+			(at 121.92 91.44 0)
+			(hide yes)
+			(show_name no)
+			(do_not_autoplace no)
+			(effects
+				(font
+					(size 1.27 1.27)
+				)
+			)
+		)
+		(property "Description" "Resistor"
+			(at 121.92 91.44 0)
+			(hide yes)
+			(show_name no)
+			(do_not_autoplace no)
+			(effects
+				(font
+					(size 1.27 1.27)
+				)
+			)
+		)
+		(pin "2"
+		)
+		(pin "1"
+		)
+		(instances
+			(project "1ST_Schematix"
+				(path "/59c2502d-7c28-4023-9b54-15ec9e15e6d4/58991d82-9dd2-4511-b974-9bfcbd0b4f51"
+					(reference "R11")
+					(unit 1)
+				)

Commit message: Update KiCad + Création Soft_Inhibot.ioc
Soft_Inhibot est mieux que juste Software. C'est mon avis...
Parts:
- added D3: 3.3V, Package_DFN_QFN:Texas_RTW_WQFN-24-1EP_4x4mm_P0.5mm_EP2.7x2.7mm_ThermalVias, symbol Device:LED
- added R13: 4.7k, Resistor_SMD:R_0402_1005Metric, symbol Device:R_Small
- R5: value R -> 10k
Connections:
- net +3.3V: now also D3.2 (A)
- net GND: now also R13.2
- new net: D3.1 (K), R13.1
Other:
- title: (none) -> Inhibot
- moved on the sheet: D1, D2, R6, R7

Commit message: Update PCB
Parts:
- removed D3: 3.3V, Package_DFN_QFN:Texas_RTW_WQFN-24-1EP_4x4mm_P0.5mm_EP2.7x2.7mm_ThermalVias, symbol Device:LED
- removed R13: 4.7k, Resistor_SMD:R_0402_1005Metric, symbol Device:R_Small

Commit message: Power Update Kicad
Parts:
- added C18, C19: C, symbol Device:C
- added C20: 1u, symbol Device:C
- added D3: D, Diode_THT:Diode_Bridge_IXYS_GUFP, symbol Device:D
- added Q1: DMP1045U-7, Package_TO_SOT_SMD:SOT-23, symbol Transistor_FET:DMP3099L
- added Q2: MMDT2222A, Package_TO_SOT_SMD:SOT-363_SC-70-6, symbol Transistor_BJT:MMDT2222A
- added R13, R18: 100k, Package_TO_SOT_SMD:SOT-363_SC-70-6, symbol Device:R_Small
- added R19, R20: 10k, symbol Device:R
- added U7: BQ27220YZFR, Package_BGA:Texas_DSBGA-9_1.4715x1.4715mm_Layout3x3_P0.5mm, symbol inhibot_lib:BQ27220YZFR
Connections:
- net +3.3V: now also R19.1
- net +5V: no longer C7.1, U3.1 (VIN), U3.3 (ON/~{OFF})
- net BMS_SCL: now also U7.A2 (SDA)
- net BMS_SDA: now also U7.A3 (SCL)
- net GND: now also C18.2, C19.2, C20.2, R13.2, R18.2, R20.2, U7.B2 (VSS)
- net VBAT: now also C7.1, U3.1 (VIN), U3.3 (ON/~{OFF})
- net USB_5V: now reaches C1.1, J1.A4 (VBUS), J1.A9 (VBUS), J1.B4 (VBUS), J1.B9 (VBUS), U4.5 (VBUS)
- net USB_5V: now also D3.1 (K), Q1.3 (D), Q2.4 (E2); no longer U2.1 (VBUS)
- new net: Q1.1 (G), Q2.1 (E1), R18.1
- new net: D3.2 (A), Q2.2 (B1), Q2.3 (C2), Q2.5 (B2), R13.1
- new net: C18.1, C19.1, U7.B3 (VDD)
- new net: R20.1, U7.B1 (BIN)
- new net: R19.2, U7.A1 (GPOUT)
- new net: C20.1, U7.C3 (BAT)
- new net VBUS: Q1.2 (S), Q2.6 (C1), U2.1 (VBUS)
Other:
- moved on the sheet: C1, C10, C11, C2, C3, C4, C5, C6, C7, C8, C9, D1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

Commit message: nom des compo
Parts:
- renumbered C1 to C301, C18 to C302, C19 to C303, C4 to C304, C5 to C305, C3 to C306, C10 to C307, C2 to C308, C11 to C309, C6 to C310, C20 to C311, C7 to C312, C9 to C313, C8 to C314, D3 to D301, D1 to D302, D2 to D303, J1 to J301, L1 to L301, Q2 to Q301, Q1 to Q302, R13 to R301, R1 to R302, R2 to R303, R18 to R304, R12 to R305, R11 to R306, R19 to R307, R5 to R308, R4 to R309, R3 to R310, R20 to R311, R6 to R312, R7 to R313, U4 to U301, U2 to U302, U7 to U303, U3 to U304
