File: Hardware/1ST_Schematix/Sensor_Inhibot.kicad_sch (KiCad schematic)
At the start: 0 parts

Commit message: Sensor PCB
Parts:
- added C12, C13: 100n, Package_SO:SOIC-16_3.9x9.9mm_P1.27mm, symbol Device:C_Small
- added R10, R8, R9: 1k, Resistor_SMD:R_0402_1005Metric, symbol Device:R_Small
- added U5: LSM6DSL, Package_LGA:LGA-14_3x2.5mm_P0.5mm_LayoutBorder3x4y, symbol Sensor_Motion:LSM6DSL
Connections:
- new net: R9.2, U5.3 (SCX)
- new net: R10.2, U5.12 (CS)
- new net: R8.2, U5.2 (SDX)
- new net +3.3V: C12.1, C13.1, R10.1, U5.5 (VDDIO), U5.8 (VDD)
- new net GND: C12.2, C13.2, R8.1, R9.1, U5.6 (GND), U5.7 (GND)
- new net INT1_Mag: U5.4 (INT1)
- new net INT2_Mag: U5.9 (INT2)
- new net SCL_Mag: U5.13 (SCL)
- new net SDA_Mag: U5.14 (SDA)
- no-connect marks 0 -> 1

Commit message: Update KiCad + Création Soft_Inhibot.ioc
Soft_Inhibot est mieux que juste Software. C'est mon avis...
Parts:
- added C14: 10p, Package_SO:TSSOP-16_4.4x5mm_P0.65mm, symbol Device:C_Small
- added C15: 2.2u, symbol Device:C_Small
- added R14: 200m, Resistor_THT:R_Array_SIP4, symbol Device:R_Small
- added U6: DRV8833PW, Package_SO:TSSOP-16_4.4x5mm_P0.65mm, symbol Driver_Motor:DRV8833PW
Connections:
- net GND: now also C15.1, R14.1, U6.13 (GND)
- new net: C15.2, U6.14 (VINT)
- new net: C14.1, U6.11 (VCP)
- new net: R14.2, U6.3 (AISEN), U6.6 (BISEN)
- new net AOUT1: U6.2 (AOUT1)
- new net AOUT2: U6.4 (AOUT2)
- new net BOUT1: U6.7 (BOUT1)
- new net BOUT2: U6.5 (BOUT2)
- new net PWM1: U6.16 (AIN1)
- new net PWM2: U6.15 (AIN2)
- new net PWM3: U6.9 (BIN1)
- new net PWM4: U6.10 (BIN2)
- new net VM: C14.2, U6.12 (VM)
Other:
- title: (none) -> Inhibot
- moved on the sheet: C12, C13, R10, R8, R9, U5

Commit message: Update PCB
Parts:
- added C17: 10u, symbol Device:C_Small
Connections:
- net GND: now also C17.1
- net VM: now also U6.1 (~{SLEEP}), C17.2
Other:
- moved on the sheet: C15

Commit message: nom des compo
Parts:
- renumbered C12 to C401, C13 to C402, C14 to C403, C15 to C404, C17 to C405, R8 to R401, R9 to R402, R10 to R403, R14 to R404, U5 to U401, U6 to U402
Changed lines of the file:
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@@
 		(in_pos_files yes)
 		(dnp no)
-		(property "Reference" "R9"
+		(property "Reference" "R402"
 			(at 63.5 94.742 90)
 			(show_name no)
@@
 			(project "1ST_Schematix"
 				(path "/59c2502d-7c28-4023-9b54-15ec9e15e6d4/bf29c48a-0938-4b44-b61a-f77bea55e593"
-					(reference "R9")
+					(reference "R402")
 					(unit 1)
 				)
@@
 		(dnp no)
 		(fields_autoplaced yes)
-		(property "Reference" "#PWR021"
+		(property "Reference" "#PWR0406"
 			(at 95.25 74.93 0)
 			(hide yes)
@@
 			(project "1ST_Schematix"
 				(path "/59c2502d-7c28-4023-9b54-15ec9e15e6d4/bf29c48a-0938-4b44-b61a-f77bea55e593"
-					(reference "#PWR021")
+					(reference "#PWR0406")
 					(unit 1)
 				)
@@
 		(in_pos_files yes)
 		(dnp no)
-		(property "Reference" "C15"
+		(property "Reference" "C404"
 			(at 208.026 70.866 90)
 			(show_name no)
@@
 			(project "1ST_Schematix"
 				(path "/59c2502d-7c28-4023-9b54-15ec9e15e6d4/bf29c48a-0938-4b44-b61a-f77bea55e593"
-					(reference "C15")
+					(reference "C404")
 					(unit 1)
 				)
@@
 		(in_pos_files yes)
 		(dnp no)
-		(property "Reference" "R10"
+		(property "Reference" "R403"
 			(at 71.12 104.902 90)
 			(show_name no)
@@
 			(project "1ST_Schematix"
 				(path "/59c2502d-7c28-4023-9b54-15ec9e15e6d4/bf29c48a-0938-4b44-b61a-f77bea55e593"
-					(reference "R10")
+					(reference "R403")
 					(unit 1)
 				)
@@
 		(dnp no)
 		(fields_autoplaced yes)
-		(property "Reference" "#PWR018"
+		(property "Reference" "#PWR0403"
 			(at 85.09 74.93 0)
 			(hide yes)
@@
 			(project "1ST_Schematix"
 				(path "/59c2502d-7c28-4023-9b54-15ec9e15e6d4/bf29c48a-0938-4b44-b61a-f77bea55e593"
-					(reference "#PWR018")
+					(reference "#PWR0403")
 					(unit 1)
 				)
@@
 		(dnp no)
 		(fields_autoplaced yes)
-		(property "Reference" "U5"
+		(property "Reference" "U401"
 			(at 91.0433 110.49 0)
 			(show_name no)
@@
 			(project "1ST_Schematix"
 				(path "/59c2502d-7c28-4023-9b54-15ec9e15e6d4/bf29c48a-0938-4b44-b61a-f77bea55e593"
-					(reference "U5")
+					(reference "U401")
 					(unit 1)
 				)
@@
 		(in_pos_files yes)
 		(dnp no)
-		(property "Reference" "C17"
+		(property "Reference" "C405"
 			(at 220.726 80.264 90)
 			(show_name no)
@@
 			(project "1ST_Schematix"
 				(path "/59c2502d-7c28-4023-9b54-15ec9e15e6d4/bf29c48a-0938-4b44-b61a-f77bea55e593"
-					(reference "C17")
+					(reference "C405")
 					(unit 1)
 				)
@@
 		(in_pos_files yes)
 		(dnp no)
-		(property "Reference" "#PWR017"
+		(property "Reference" "#PWR0402"
 			(at 59.69 106.68 0)
 			(hide yes)
@@
 			(project "1ST_Schematix"
 				(path "/59c2502d-7c28-4023-9b54-15ec9e15e6d4/bf29c48a-0938-4b44-b61a-f77bea55e593"
-					(reference "#PWR017")
+					(reference "#PWR0402")
 					(unit 1)
 				)
@@
 		(dnp no)
 		(fields_autoplaced yes)
-		(property "Reference" "#PWR044"
+		(property "Reference" "#PWR0411"
 			(at 223.52 88.9 0)
 			(hide yes)
@@
 			(project "1ST_Schematix"
 				(path "/59c2502d-7c28-4023-9b54-15ec9e15e6d4/bf29c48a-0938-4b44-b61a-f77bea55e593"
-					(reference "#PWR044")
+					(reference "#PWR0411")
 					(unit 1)
 				)
@@
 		(in_pos_files yes)
 		(dnp no)
-		(property "Reference" "R8"
+		(property "Reference" "R401"
 			(at 63.5 88.392 90)
 			(show_name no)
@@
 			(project "1ST_Schematix"
 				(path "/59c2502d-7c28-4023-9b54-15ec9e15e6d4/bf29c48a-0938-4b44-b61a-f77bea55e593"
-					(reference "R8")
+					(reference "R401")
 					(unit 1)
 				)
@@
 		(dnp no)
 		(fields_autoplaced yes)
-		(property "Reference" "#PWR016"
+		(property "Reference" "#PWR0401"
 			(at 59.69 100.33 0)
 			(hide yes)
@@
 			(project "1ST_Schematix"
 				(path "/59c2502d-7c28-4023-9b54-15ec9e15e6d4/bf29c48a-0938-4b44-b61a-f77bea55e593"
-					(reference "#PWR016")
+					(reference "#PWR0401")
 					(unit 1)
 				)
@@
 		(dnp no)
 		(fields_autoplaced yes)
-		(property "Reference" "C14"
+		(property "Reference" "C403"
 			(at 187.96 85.0899 0)
 			(show_name no)
@@
 			(project "1ST_Schematix"
 				(path "/59c2502d-7c28-4023-9b54-15ec9e15e6d4/bf29c48a-0938-4b44-b61a-f77bea55e593"
-					(reference "C14")
+					(reference "C403")
 					(unit 1)
 				)
@@
 		(dnp no)
 		(fields_autoplaced yes)
-		(property "Reference" "#PWR028"
+		(property "Reference" "#PWR0410"
 			(at 208.28 120.65 0)
 			(hide yes)
@@
 			(project "1ST_Schematix"
 				(path "/59c2502d-7c28-4023-9b54-15ec9e15e6d4/bf29c48a-0938-4b44-b61a-f77bea55e593"
-					(reference "#PWR028")
+					(reference "#PWR0410")
 					(unit 1)
 				)
@@
 		(dnp no)
 		(fields_autoplaced yes)
-		(property "Reference" "#PWR026"
+		(property "Reference" "#PWR0408"
 			(at 184.15 104.14 0)
 			(hide yes)
@@
 			(project "1ST_Schematix"
 				(path "/59c2502d-7c28-4023-9b54-15ec9e15e6d4/bf29c48a-0938-4b44-b61a-f77bea55e593"
-					(reference "#PWR026")
+					(reference "#PWR0408")
 					(unit 1)
 				)
@@
 		(in_pos_files yes)
 		(dnp no)
-		(property "Reference" "#PWR022"
+		(property "Reference" "#PWR0407"
 			(at 95.25 83.82 0)
 			(hide yes)
@@
 			(project "1ST_Schematix"
 				(path "/59c2502d-7c28-4023-9b54-15ec9e15e6d4/bf29c48a-0938-4b44-b61a-f77bea55e593"
-					(reference "#PWR022")
+					(reference "#PWR0407")
 					(unit 1)
 				)
@@
 		(dnp no)
 		(fields_autoplaced yes)
-		(property "Reference" "U6"
+		(property "Reference" "U402"
 			(at 210.4233 114.3 0)
 			(show_name no)
@@
 			(project "1ST_Schematix"
 				(path "/59c2502d-7c28-4023-9b54-15ec9e15e6d4/bf29c48a-0938-4b44-b61a-f77bea55e593"
-					(reference "U6")
+					(reference "U402")
 					(unit 1)
 				)
@@
 		(dnp no)
 		(fields_autoplaced yes)
-		(property "Reference" "C13"
+		(property "Reference" "C402"
 			(at 97.79 73.6599 0)
 			(show_name no)
@@
 			(project "1ST_Schematix"
 				(path "/59c2502d-7c28-4023-9b54-15ec9e15e6d4/bf29c48a-0938-4b44-b61a-f77bea55e593"
-					(reference "C13")
+					(reference "C402")
 					(unit 1)
 				)
@@
 		(in_pos_files yes)
 		(dnp no)
-		(property "Reference" "#PWR019"
+		(property "Reference" "#PWR0404"
 			(at 85.09 83.82 0)
 			(hide yes)
@@
 			(project "1ST_Schematix"
 				(path "/59c2502d-7c28-4023-9b54-15ec9e15e6d4/bf29c48a-0938-4b44-b61a-f77bea55e593"
-					(reference "#PWR019")
+					(reference "#PWR0404")
 					(unit 1)
 				)
@@
 		(in_pos_files yes)
 		(dnp no)
-		(property "Reference" "R14"
+		(property "Reference" "R404"
 			(at 189.23 94.488 90)
 			(show_name no)
@@
 			(project "1ST_Schematix"
 				(path "/59c2502d-7c28-4023-9b54-15ec9e15e6d4/bf29c48a-0938-4b44-b61a-f77bea55e593"
-					(reference "R14")
+					(reference "R404")
 					(unit 1)
 				)
@@
 		(dnp no)
 		(fields_autoplaced yes)
-		(property "Reference" "#PWR020"
+		(property "Reference" "#PWR0405"
 			(at 88.9 116.84 0)
 			(hide yes)
@@
 			(project "1ST_Schematix"
 				(path "/59c2502d-7c28-4023-9b54-15ec9e15e6d4/bf29c48a-0938-4b44-b61a-f77bea55e593"
-					(reference "#PWR020")
+					(reference "#PWR0405")
 					(unit 1)
 				)
@@
 		(dnp no)
 		(fields_autoplaced yes)
-		(property "Reference" "#PWR027"
+		(property "Reference" "#PWR0409"
 			(at 203.2 81.28 0)
 			(hide yes)
@@
 			(project "1ST_Schematix"
 				(path "/59c2502d-7c28-4023-9b54-15ec9e15e6d4/bf29c48a-0938-4b44-b61a-f77bea55e593"
-					(reference "#PWR027")
+					(reference "#PWR0409")
 					(unit 1)
 				)
@@
 		(in_pos_files yes)
 		(dnp no)
-		(property "Reference" "C12"
+		(property "Reference" "C401"
 			(at 80.01 73.66 0)
 			(show_name no)
@@
 			(project "1ST_Schematix"
 				(path "/59c2502d-7c28-4023-9b54-15ec9e15e6d4/bf29c48a-0938-4b44-b61a-f77bea55e593"
-					(reference "C12")
-					(unit 1)
-				)
+					(reference "C401")
+					(unit 1)
+				)

Commit message: Bus I2C2
Parts:
- C401, C402: footprint Package_SO:SOIC-16_3.9x9.9mm_P1.27mm -> Capacitor_SMD:C_0402_1005Metric
- C403: footprint Package_SO:TSSOP-16_4.4x5mm_P0.65mm -> Capacitor_SMD:C_0402_1005Metric
- C404, C405: footprint (none) -> Capacitor_SMD:C_0402_1005Metric
Changed lines of the file:
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@@
 			)
 		)
-		(property "Footprint" ""
+		(property "Footprint" "Capacitor_SMD:C_0402_1005Metric"
 			(at 208.28 73.66 0)
 			(hide yes)
@@
 			)
 		)
-		(property "Footprint" ""
+		(property "Footprint" "Capacitor_SMD:C_0402_1005Metric"
 			(at 223.52 80.01 0)
 			(hide yes)
@@
 			)
 		)
-		(property "Footprint" "Package_SO:TSSOP-16_4.4x5mm_P0.65mm"
+		(property "Footprint" "Capacitor_SMD:C_0402_1005Metric"
 			(at 185.42 86.36 0)
 			(hide yes)
@@
 			)
 		)
-		(property "Footprint" "Package_SO:SOIC-16_3.9x9.9mm_P1.27mm"
+		(property "Footprint" "Capacitor_SMD:C_0402_1005Metric"
 			(at 95.25 74.93 0)
 			(hide yes)
@@
 			)
 		)
-		(property "Footprint" "Package_SO:SOIC-16_3.9x9.9mm_P1.27mm"
+		(property "Footprint" "Capacitor_SMD:C_0402_1005Metric"
 			(at 85.09 74.93 0)
 			(hide yes)

Commit message: Update before INT
Parts:
- added R405, R406: 1k, Resistor_THT:R_Array_SIP4, symbol Device:R_Small
Connections:
- net at U402.8 (~{FAULT}): now also R406.1
- net VM renamed +5V
- net +5V: now also R405.2, R406.2; no longer U402.1 (~{SLEEP})
- new net: R405.1, U402.1 (~{SLEEP})
