File: Hardware/1ST_Schematix/Connector_Inhibot.kicad_sch (KiCad schematic)
At the start: 7 parts, among them J2 Conn_01x02, J3 Conn_01x03, J4 Conn_01x06, J5 Conn_01x06, J6 Conn_01x03

Commit message: Update PCB
Parts:
- added J10: Conn_01x05, Package_DFN_QFN:QFN-20-1EP_5x5mm_P0.65mm_EP3.35x3.35mm, symbol Connector_Generic:Conn_01x05
- added J11: Conn_01x03, symbol Connector_Generic:Conn_01x03
- added J7, J8, J9: Conn_01x06, symbol Connector_Generic:Conn_01x06
- added JP3, JP4: SolderJumper_2_Open, Jumper:SolderJumper-2_P1.3mm_Open_TrianglePad1.0x1.5mm, symbol Jumper:SolderJumper_2_Open
Connections:
- net +3.3V: now also J10.1 (Pin_1), J7.1 (Pin_1), J8.1 (Pin_1), J9.1 (Pin_1)
- net +5V: now also J6.2 (Pin_2); no longer J6.1 (Pin_1)
- net GND: now also J10.2 (Pin_2), J11.3 (Pin_3), J7.6 (Pin_6), J8.2 (Pin_2), J9.2 (Pin_2)
- net Servomot: now also J6.1 (Pin_1); no longer J6.2 (Pin_2)
- new net: J11.1 (Pin_1), JP3.1 (A)
- new net: J11.2 (Pin_2), JP4.1 (A)
- new net INT1_Mag: J7.4 (Pin_4)
- new net INT2_Mag: J7.5 (Pin_5)
- new net INT_Color: J10.5 (Pin_5)
- new net RX_Bluetooth: JP3.2 (B)
- new net SCL_Color: J10.3 (Pin_3)
- new net SCL_Mag_conn: J7.3 (Pin_3)
- new net SCL_TOF: J8.3 (Pin_3), J9.3 (Pin_3)
- new net SDA_Color: J10.4 (Pin_4)
- new net SDA_Mag_conn: J7.2 (Pin_2)
- new net SDA_TOF: J8.4 (Pin_4), J9.4 (Pin_4)
- new net TOF1_GPIO1: J9.5 (Pin_5)
- new net TOF1_XST: J9.6 (Pin_6)
- new net TOF2_GPIO1: J8.5 (Pin_5)
- new net TOF2_XST: J8.6 (Pin_6)
- new net TX_Bluetooth: JP4.2 (B)

Commit message: nom des compo
Parts:
- renumbered C16 to C501, D4 to D501, J4 to J501, J2 to J502, J5 to J503, J10 to J504, J3 to J505, J6 to J506, J11 to J507, J7 to J508, J9 to J509, J8 to J510, JP3 to JP501, JP4 to JP502

Commit message: Bus I2C2
Parts:
- C501: footprint (none) -> Capacitor_SMD:C_0402_1005Metric
Changed lines of the file:
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@@
 			)
 		)
-		(property "Footprint" ""
+		(property "Footprint" "Capacitor_SMD:C_0402_1005Metric"
 			(at 149.86 46.99 0)
 			(hide yes)

Commit message: Update before INT
Parts:
- added H501_OUT, H502_OUT: MountingHole_Pad, Module:Maple_Mini, symbol Mechanical:MountingHole_Pad
- added J511_OUT: Conn_01x06, symbol Connector_Generic:Conn_01x06
Connections:
- net +3.3V: now also J511_OUT.1 (Pin_1)
- net GND: now also H501_OUT.1, H502_OUT.1, J511_OUT.6 (Pin_6)
- net INT1_Mag: now also J511_OUT.4 (Pin_4)
- net INT2_Mag: now also J511_OUT.5 (Pin_5)
- net SCL_Mag_conn: now also J511_OUT.3 (Pin_3)
- net SDA_Mag_conn: now also J511_OUT.2 (Pin_2)
Other:
- moved on the sheet: J501, J508, J510

Commit message: Update KiCad and STM32CubeMX
Ready for the check-in
Parts:
- removed C501: 1000u, Capacitor_SMD:C_0402_1005Metric, symbol Device:C_Small
- removed D501: LED_RGB, LED_SMD:LED_WS2812_PLCC6_5.0x5.0mm_P1.6mm, symbol Device:LED_RGB
- removed H501_OUT, H502_OUT: MountingHole_Pad, Module:Maple_Mini, symbol Mechanical:MountingHole_Pad
- removed J505: Conn_01x03, symbol Connector_Generic:Conn_01x03
- removed J511_OUT: Conn_01x06, symbol Connector_Generic:Conn_01x06
- added C502, C503: 100n, Capacitor_SMD:C_0402_1005Metric, symbol Device:C_Small
- added D502: WS2812B, LED_SMD:LED_WS2812B-Mini_PLCC4_3.5x3.5mm, symbol LED:WS2812B
- added J511: Conn_01x03, symbol Connector_Generic:Conn_01x03
- added U501: SN74AHCT1G125DBVR, Package_TO_SOT_SMD:SOT-23-5, symbol 74xGxx:74AHCT1G125
Connections:
- net +5V: now also C502.1, C503.2, D502.1 (VDD), J511.1 (Pin_1), U501.5 (VCC)
- net GND: now also C502.2, C503.1, D502.3 (VSS), J511.3 (Pin_3), U501.1, U501.3 (GND)
- net RGB_IN: now also U501.2
- new net: D502.2 (DOUT), J511.2 (Pin_2)
- new net NP_5V: D502.4 (DIN), U501.4
- no-connect marks 1 -> 0
Other:
- moved on the sheet: J501, J502, J503, J508

Commit message: schematic review with esteemed professor
Parts:
- removed J502: Conn_01x02, symbol Connector_Generic:Conn_01x02
- removed JP501, JP502: SolderJumper_2_Open, Jumper:SolderJumper-2_P1.3mm_Open_TrianglePad1.0x1.5mm, symbol Jumper:SolderJumper_2_Open
Connections:
- net RX_Bluetooth: now also J507.1 (Pin_1)
- net TX_Bluetooth: now also J507.2 (Pin_2)

Commit message: prints for component except 10mOhm
Parts:
- J501, J503, J508, J509, J510: footprint (none) -> Connector_JST:JST_EH_B6B-EH-A_1x06_P2.50mm_Vertical; now left out of the parts list
- J504: footprint Package_DFN_QFN:QFN-20-1EP_5x5mm_P0.65mm_EP3.35x3.35mm -> Connector_JST:JST_EH_B5B-EH-A_1x05_P2.50mm_Vertical; now left out of the parts list
- J506, J507, J511: footprint (none) -> Connector_JST:JST_EH_B3B-EH-A_1x03_P2.50mm_Vertical; now left out of the parts list
Changed lines of the file:
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@@
 		(body_style 1)
 		(exclude_from_sim no)
-		(in_bom yes)
+		(in_bom no)
 		(on_board yes)
 		(in_pos_files yes)
@@
 			)
 		)
-		(property "Footprint" ""
+		(property "Footprint" "Connector_JST:JST_EH_B6B-EH-A_1x06_P2.50mm_Vertical"
 			(at 60.96 43.18 0)
 			(hide yes)
@@
 		(body_style 1)
 		(exclude_from_sim no)
-		(in_bom yes)
+		(in_bom no)
 		(on_board yes)
 		(in_pos_files yes)
@@
 			)
 		)
-		(property "Footprint" ""
+		(property "Footprint" "Connector_JST:JST_EH_B3B-EH-A_1x03_P2.50mm_Vertical"
 			(at 142.24 93.98 0)
 			(hide yes)
@@
 		(body_style 1)
 		(exclude_from_sim no)
-		(in_bom yes)
+		(in_bom no)
 		(on_board yes)
 		(in_pos_files yes)
@@
 			)
 		)
-		(property "Footprint" ""
+		(property "Footprint" "Connector_JST:JST_EH_B6B-EH-A_1x06_P2.50mm_Vertical"
 			(at 45.72 43.18 0)
 			(hide yes)
@@
 		(body_style 1)
 		(exclude_from_sim no)
-		(in_bom yes)
+		(in_bom no)
 		(on_board yes)
 		(in_pos_files yes)
@@
 			)
 		)
-		(property "Footprint" ""
+		(property "Footprint" "Connector_JST:JST_EH_B6B-EH-A_1x06_P2.50mm_Vertical"
 			(at 233.68 97.79 0)
 			(hide yes)
@@
 		(body_style 1)
 		(exclude_from_sim no)
-		(in_bom yes)
+		(in_bom no)
 		(on_board yes)
 		(in_pos_files yes)
@@
 			)
 		)
-		(property "Footprint" ""
+		(property "Footprint" "Connector_JST:JST_EH_B6B-EH-A_1x06_P2.50mm_Vertical"
 			(at 231.14 55.88 0)
 			(hide yes)
@@
 		(body_style 1)
 		(exclude_from_sim no)
-		(in_bom yes)
+		(in_bom no)
 		(on_board yes)
 		(in_pos_files yes)
@@
 			)
 		)
-		(property "Footprint" ""
+		(property "Footprint" "Connector_JST:JST_EH_B3B-EH-A_1x03_P2.50mm_Vertical"
 			(at 147.32 137.16 0)
 			(hide yes)
@@
 		(body_style 1)
 		(exclude_from_sim no)
-		(in_bom yes)
+		(in_bom no)
 		(on_board yes)
 		(in_pos_files yes)
@@
 			)
 		)
-		(property "Footprint" ""
+		(property "Footprint" "Connector_JST:JST_EH_B6B-EH-A_1x06_P2.50mm_Vertical"
 			(at 217.17 97.79 0)
 			(hide yes)
@@
 		(body_style 1)
 		(exclude_from_sim no)
-		(in_bom yes)
+		(in_bom no)
 		(on_board yes)
 		(in_pos_files yes)
@@
 			)
 		)
-		(property "Footprint" ""
+		(property "Footprint" "Connector_JST:JST_EH_B3B-EH-A_1x03_P2.50mm_Vertical"
 			(at 186.69 52.07 0)
 			(hide yes)
@@
 		(body_style 1)
 		(exclude_from_sim no)
-		(in_bom yes)
+		(in_bom no)
 		(on_board yes)
 		(in_pos_files yes)
@@
 			)
 		)
-		(property "Footprint" "Package_DFN_QFN:QFN-20-1EP_5x5mm_P0.65mm_EP3.35x3.35mm"
+		(property "Footprint" "Connector_JST:JST_EH_B5B-EH-A_1x05_P2.50mm_Vertical"
 			(at 80.01 134.62 0)
 			(hide yes)
