File: Hardware/1ST_Schematix/Connector_Inhibot.kicad_sch (KiCad schematic)
At the start: 22 parts, among them J501 Conn_01x06, J502 Conn_01x03, J503 Conn_01x06, J504 Conn_01x05, J506 Conn_01x03, J507 Conn_01x03, J508 Conn_01x06, J509 Conn_01x06, J510 Conn_01x06, J511 Conn_01x03, U501 SN74AHCT1G125DBVR

Commit message: commande ready
Parts:
- D502: JLCPCB Parts # C527089 -> C52941386
Changed lines of the file:
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@@
 			)
 		)
-		(property "JLCPCB Parts #" "C527089"
+		(property "JLCPCB Parts #" "C52941386"
 			(at 158.75 52.07 0)
 			(hide yes)
