File: Hardware/1ST_Schematix/1ST_Schematix.kicad_pcb (KiCad board)
At the start: 4 copper layers, 99.9 x 99.9 mm, 110 parts, among them J201 Conn_ST_STDC14, J301 USB_C_Receptacle_USB2.0_16P, J302 Conn_01x02, J501 Conn_01x06, J503 Conn_01x06, J504 Conn_01x05, J506 Conn_01x03, J507 Conn_01x03, J508 Conn_01x06, J509 Conn_01x06, J510 Conn_01x06, J511 Conn_01x03, J511_OUT401 Conn_01x06, Q301 MMDT2222A, Q302 DMP1045U-7, Q303 DMN313DLT-7, SW101 SW_Push, SW201 SW_Push, U201 STM32G431RBTx, U301 USBLC6-2SC6, U302 BQ25896RTW, U303 BQ27220YZFR, U305 BU33SD5WG-TR, U401 LSM6DSL, U402 DRV8833PW, U501 SN74AHCT1G125DBVR, Y201 X322516MLB4SI

Commit message: midway
Parts:
- L301: footprint Package_SO:SOIC-16_3.9x9.9mm_P1.27mm -> Inductor_SMD:L_0603_1608Metric
- moved TP304 203.0 mm to (240.6, 119.9)
- moved TP303 202.5 mm to (236.9, 129.5)
- moved TP305 194.2 mm to (235.5, 74.5)
- moved TP302 192.9 mm to (230.7, 110.1)
- moved TP301 183.7 mm to (216.7, 123.5)
- moved C302 151.1 mm to (190.4, 122.0), turned to -90 degrees
- moved C303 149.5 mm to (189.3, 122.0), turned to -90 degrees
- moved C311 147.9 mm to (190.6, 127.0), turned to -90 degrees
- moved JP301 147.4 mm to (185.0, 136.0), turned to 180 degrees
- moved J302 144.4 mm to (195.2, 125.8), turned to 90 degrees
- moved U301 141.5 mm to (186.1, 110.5), turned to 180 degrees
- moved R303 139.4 mm to (190.0, 111.5), turned to 180 degrees
- moved R302 139.2 mm to (190.0, 108.5), turned to 180 degrees
- moved SW101 138.9 mm to (186.0, 129.1), turned to 180 degrees
- moved L301 137.1 mm to (174.9, 123.4), turned to -90 degrees
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Routing:
- net /SDA1: track 0.00 -> 90.2 mm
- net /SCL1: track 0.00 -> 82.8 mm
- net /Power/STM32_D+: track 0.00 -> 77.0 mm
- net /Power/STM32_D-: track 0.00 -> 75.8 mm
- net /Connectors/RX_Bluetooth: track 0.00 -> 42.9 mm
- net /Connectors/TX_Bluetooth: track 0.00 -> 39.8 mm
- net /STM32/FAULT: track 1.60 -> 36.7 mm, vias 0 -> 2
- net /TOF2_GPIO: track 0.00 -> 34.1 mm
- net /TOF2_XST: track 0.00 -> 27.5 mm
- net /Connectors/INT1_Mag: track 0.00 -> 26.2 mm
- net /Connectors/INT2_Mag: track 0.00 -> 25.4 mm
- net Net-(JP301-A): track 0.00 -> 18.0 mm
- net /Power/~{QON}: track 0.00 -> 17.5 mm, vias 0 -> 1
- net GND: track 0.00 -> 9.56 mm, vias 0 -> 9
- net /Power/USB_D-: track 0.00 -> 8.17 mm
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- added copper zone on F.Cu, net +BATT
Other:
- board size 99.9 x 99.9 mm -> 100 x 99.7 mm

Commit message: routage à faire vérifier
Parts:
- added J502: Conn_01x03, Connector_JST:JST_EH_B3B-EH-A_1x03_P2.50mm_Vertical, F.Cu at (106.0, 118.5)
- C302: footprint Capacitor_SMD:C_0402_1005Metric -> Capacitor_SMD:C_0603_1608Metric
- C310: footprint Capacitor_SMD:C_0402_1005Metric -> Capacitor_SMD:C_1206_3216Metric
- moved D202 173.1 mm to (193.2, 102.0), turned to 180 degrees
- moved R203 166.9 mm to (193.4, 103.5)
- moved R202 162.6 mm to (195.3, 119.3)
- moved D201 162.4 mm to (195.3, 117.8), turned to 180 degrees
- moved C301 145.5 mm to (187.7, 107.3), turned to 90 degrees
- moved R207 136.3 mm to (161.2, 108.3), turned to 90 degrees
- moved R208 133.2 mm to (164.0, 124.4)
- moved R205 123.4 mm to (132.2, 86.2), turned to 90 degrees
- moved R206 122.5 mm to (128.4, 86.5), turned to 180 degrees
- moved C305 113.8 mm to (170.2, 120.0), turned to 180 degrees
- moved J511 101.3 mm to (106.0, 107.2), turned to -90 degrees
- moved TP305 95.8 mm to (170.1, 144.4)
- moved J506 95.1 mm to (106.0, 129.7), turned to -90 degrees
- moved C503 90.3 mm to (115.0, 111.2), turned to 90 degrees
- moved D502 86.6 mm to (112.4, 108.6)
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Connections:
- J506 pad 1: /Connectors/Servomot -> /Connectors/Servomot2
- U201 pad 20: /Connectors/Servomot -> /Connectors/Servomot1
- U201 pad 21: /Connectors/Servomot -> /Connectors/Servomot2
Routing:
- net /Connectors/2_Encoder_A: track 0.00 -> 84.9 mm, vias 0 -> 2
- net /Connectors/2_Encoder_B: track 0.00 -> 83.3 mm, vias 0 -> 2
- net /TOF1_GPIO: track 0.00 -> 68.7 mm, vias 0 -> 1
- net /TOF1_XST: track 0.00 -> 67.3 mm, vias 0 -> 1
- net /Power/SYS: track 0.00 -> 62.8 mm, vias 0 -> 2
- net /BMS_SDA: track 0.10 -> 62.6 mm, vias 0 -> 2
- net /BMS_SCL: track 0.00 -> 61.9 mm
- net /Connectors/Servomot2: track 0.00 -> 54.6 mm, vias 0 -> 1
- net /Connectors/Servomot1: track 0.00 -> 52.1 mm, vias 0 -> 1
- net /STM32/LED_STATUS: track 0.00 -> 45.4 mm, vias 0 -> 2
- net /Power/~{QON}: track 17.5 -> 57.1 mm, vias 1 -> 2
- net /Power/STM32_D+: track 77.0 -> 39.0 mm
- net /Power/STM32_D-: track 75.8 -> 39.6 mm
- net /Power/BMS_~{INT}: track 0.00 -> 35.0 mm
- net Net-(JP301-A): track 18.0 -> 52.2 mm
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- added copper zone on In2.Cu, net +5V
- added copper zone on F.Cu, net /Power/VBAT_TO_SHUNT
- added copper zone on F.Cu, net Net-(JP302-A)

Commit message: fin du routage, plus qu'à faire le jlcpb
Parts:
- added C501: 1u, Capacitor_SMD:C_0402_1005Metric, F.Cu at (109.0, 122.4)
- added C504: 1u, Capacitor_SMD:C_0402_1005Metric, F.Cu at (109.0, 133.7)
- added C505: 100n, Capacitor_SMD:C_0402_1005Metric, F.Cu at (147.5, 83.0)
- added C506: 100n, Capacitor_SMD:C_0402_1005Metric, F.Cu at (144.8, 140.3)
- added C507: 100n, Capacitor_SMD:C_0402_1005Metric, F.Cu at (123.4, 140.3)
- added C508: 100n, Capacitor_SMD:C_0402_1005Metric, F.Cu at (109.2, 87.8)
- added C509: 100n, Capacitor_SMD:C_0402_1005Metric, F.Cu at (134.2, 83.3)
- added C510: 100n, Capacitor_SMD:C_0402_1005Metric, F.Cu at (169.7, 83.5)
- added G***: LOGO, LOGO, F.Cu at (185.6, 92.1)
- C302: footprint Capacitor_SMD:C_0603_1608Metric -> Capacitor_SMD:C_0402_1005Metric
- C310: footprint Capacitor_SMD:C_1206_3216Metric -> Capacitor_SMD:C_0402_1005Metric
- L301: footprint Inductor_SMD:L_0603_1608Metric -> Inductor_SMD:L_0402_1005Metric
- U402: footprint Package_SO:TSSOP-16_4.4x5mm_P0.65mm -> Package_SO:TSSOP-16-1EP_4.4x5mm_P0.65mm_EP3x3mm
- moved C406 9.06 mm to (148.4, 117.5)
- moved L301 2.29 mm to (173.9, 121.4), turned to 0 degrees
- moved C310 1.68 mm to (167.7, 120.1), turned to 90 degrees
- moved C306 0.94 mm to (176.3, 125.7)
- moved C503 0.76 mm to (115.1, 112.0)
- moved C308 0.74 mm to (177.4, 125.7)
- moved U402 0.10 mm to (145.3, 130.2)
- moved R404 0.06 mm to (150.1, 130.3)
- moved R407 0.06 mm to (140.4, 130.3)
- moved TP302 0.06 mm to (180.6, 144.5)
- moved TP304 0.06 mm to (177.2, 144.5)
- moved C209 0.06 mm to (138.2, 106.1)
- moved C302 0.06 mm to (191.1, 121.4)
- moved C305 0.06 mm to (170.2, 119.9)
- moved C312 0.06 mm to (176.0, 120.7)
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Routing:
- net Net-(JP301-A): track 52.2 -> 6.28 mm, vias 0 -> 5
- net +3.3V: track 48.5 -> 80.1 mm, vias 18 -> 19
- net GND: track 20.1 -> 38.9 mm, vias 26 -> 219
- net VBUS: track 23.0 -> 7.24 mm
- net +BATT: track 1.12 -> 9.91 mm
- net Net-(C304-Pad2): track 6.83 -> 0.00 mm
- net /Power/VBAT_TO_SHUNT: track 22.4 -> 28.4 mm
- net /Connectors/2_Encoder_A: track 84.9 -> 81.8 mm
- net /STM32/RCC_OSC_OUT: track 6.86 -> 8.80 mm
- net /STM32/Prog_Rx: track 16.3 -> 17.0 mm
- net /Sensors&Driver/INT1_Mag_OUT: track 15.4 -> 16.1 mm
- net /Power/STM32_D+: track 39.0 -> 39.6 mm
- net Net-(U402-AISEN): track 4.65 -> 5.24 mm
- net Net-(U402-BISEN): track 4.49 -> 5.00 mm
- net +5V: track 29.9 -> 29.6 mm, vias 3 -> 4
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- added copper zone on In1.Cu, net +5V
- added copper zone on In2.Cu, net GND
- added copper zone on F.Cu, net Net-(C304-Pad2)
- added copper zone on In1.Cu, net Net-(JP301-A)
- added copper zone on B.Cu, net VBUS
- removed copper zone on In2.Cu, net +5V
Other:
- board size 100 x 99.7 mm -> 99.9 x 99.7 mm
- board text added: "Bluetooth"
- board text added: "Color Sensor"
- board text added: "Gyro+Acc"
- board text added: "Léonard NAVIZET Bradley SERAPHIN Lucas BOISBOURDIN"
- board text added: "Moteur1"
- board text added: "Moteur2"
- board text added: "RGB Neopixel"
- board text added: "SERVO1"
- board text added: "SERVO2"
- board text added: "TOF1"
- board text added: "TOF2"

Commit message: gerber and starting jlcpcb
Parts:
- C302: footprint Capacitor_SMD:C_0402_1005Metric -> Capacitor_SMD:C_0603_1608Metric
- C310: footprint Capacitor_SMD:C_0402_1005Metric -> Capacitor_SMD:C_1206_3216Metric
- R317: value 4k7 -> 4.7k
- U201: value STM32G431RBTx -> STM32G431RBT6
- U302: value BQ25896RTW -> BQ25896RTWR
- U402: value DRV8833PW -> DRV8833PW-PR
- moved C310 5.03 mm to (172.2, 117.9), turned to 0 degrees
- moved C305 3.17 mm to (173.4, 119.9)
- moved JP303 0.15 mm to (167.8, 117.9)
- moved C302 0.12 mm to (191.2, 121.3)
Routing:
- net Net-(U302-PMID): track 2.09 -> 5.70 mm
- net /Power/REGN: track 14.6 -> 17.0 mm
- net GND: vias 219 -> 215
Other:
- board text added: "Inhibot Léonard NAVIZET Bradley SERAPHIN Lucas BOISBOURDIN"
- board text removed: "Léonard NAVIZET Bradley SERAPHIN Lucas BOISBOURDIN"

Commit message: commande ready
Routing:
- net GND: track 38.9 -> 37.7 mm
- net (no net): vias 1 -> 0
Changed lines of the file:
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@@
 		(35 "F.Fab" user)
 		(33 "B.Fab" user)
-		(39 "User.1" user)
+		(39 "User.1" user "V-Cut")
 		(41 "User.2" user)
 		(43 "User.3" user)
@@
 		(capping no)
 		(filling no)
+		(zone_defaults)
 		(pcbplotparams
 			(layerselection 0x00000000_00000000_55555555_5755f5ff)
@@
 	(gr_line
 		(start 110.05 70.063005)
-		(end 124.010495 70.063005)
+		(end 171.849495 70.0625)
 		(stroke
 			(width 0.05)
@@
 		)
 	)
-	(via
-		(at 190.51 59.4625)
-		(size 0.5)
-		(drill 0.3)
-		(layers "F.Cu" "B.Cu")
-		(net "")
+	(dimension
+		(type orthogonal)
+		(layer "F.SilkS")
+		(pts
+			(xy 200.2 138.7) (xy 100.1 138.8)
+		)
+		(height 17.1)
+		(orientation 0)
+		(format
+			(prefix "")
+			(suffix "")
+			(units 3)
+			(units_format 0)
+			(precision 4)
+			(suppress_zeroes yes)
+		)
+		(style
+			(thickness 0.1)
+			(arrow_length 1.27)
+			(text_position_mode 0)
+			(arrow_direction outward)
+			(extension_height 0.58642)
+			(extension_offset 0.5)
+			(keep_text_aligned yes)
+		)
+		(gr_text "100,1"
+			(at 150.15 154.7 0)
+			(layer "F.SilkS")
+			(effects
+				(font
+					(size 1 1)
+					(thickness 0.1)
+				)
+			)
+		)
+	)
+	(dimension
+		(type orthogonal)
+		(layer "F.SilkS")
+		(pts
+			(xy 109.3 149.9) (xy 112.7 70)
+		)
+		(height -14)
+		(orientation 1)
+		(format
+			(prefix "")
+			(suffix "")
+			(units 3)
+			(units_format 0)
+			(precision 4)
+			(suppress_zeroes yes)
+		)
+		(style
+			(thickness 0.1)
+			(arrow_length 1.27)
+			(text_position_mode 0)
+			(arrow_direction outward)
+			(extension_height 0.58642)
+			(extension_offset 0.5)
+			(keep_text_aligned yes)
+		)
+		(gr_text "79,9"
+			(at 94.2 109.95 90)
+			(layer "F.SilkS")
+			(effects
+				(font
+					(size 1 1)
+					(thickness 0.1)
+				)
+			)
+		)
 	)
 	(segment
@@
 	)
 	(segment
-		(start 170.95 123.4625)
-		(end 169.776881 123.4625)
-		(width 0.7)
-		(layer "F.Cu")
-		(net "GND")
-	)
-	(segment
 		(start 141.311698 93.8625)
 		(end 141.8 94.350802)
@@
 	)
 	(segment
-		(start 186.66 121.291881)
-		(end 189.19 121.291881)
-		(width 0.1)
-		(layer "F.Cu")
-		(net "Net-(U303-VDD)")
-	)
-	(segment
-		(start 190.349381 121.436881)
-		(end 191.05 122.1375)
-		(width 0.2)
-		(layer "F.Cu")
-		(net "Net-(U303-VDD)")
-	)
-	(segment
-		(start 189.19 121.291881)
-		(end 189.335 121.436881)
-		(width 0.2)
-		(layer "F.Cu")
-		(net "Net-(U303-VDD)")
-	)
-	(segment
-		(start 189.335 121.436881)
-		(end 190.349381 121.436881)
-		(width 0.2)
-		(layer "F.Cu")
-		(net "Net-(U303-VDD)")
-	)
-	(segment
 		(start 143.025 133.1625)
 		(end 143.1 133.0875)
@@
 	)
 	(segment
+		(start 186.66 121.291881)
+		(end 189.19 121.291881)
+		(width 0.1)
+		(layer "F.Cu")
+		(net "Net-(U303-VDD)")
+	)
+	(segment
+		(start 190.349381 121.436881)
+		(end 191.05 122.1375)
+		(width 0.2)
+		(layer "F.Cu")
+		(net "Net-(U303-VDD)")
+	)
+	(segment
+		(start 189.19 121.291881)
+		(end 189.335 121.436881)
+		(width 0.2)
+		(layer "F.Cu")
+		(net "Net-(U303-VDD)")
+	)
+	(segment
+		(start 189.335 121.436881)
+		(end 190.349381 121.436881)
+		(width 0.2)
+		(layer "F.Cu")
+		(net "Net-(U303-VDD)")
+	)
+	(segment
