File: Hardware/1ST_Schematix/_restore_backup_2026-10-05T08-37-58-085/1ST_Schematix.kicad_pcb (KiCad board)
At the start: 4 copper layers, 99.9 x 99.9 mm, 110 parts, among them J201 Conn_ST_STDC14, J301 USB_C_Receptacle_USB2.0_16P, J302 Conn_01x02, J501 Conn_01x06, J503 Conn_01x06, J504 Conn_01x05, J506 Conn_01x03, J507 Conn_01x03, J508 Conn_01x06, J509 Conn_01x06, J510 Conn_01x06, J511 Conn_01x03, J511_OUT401 Conn_01x06, Q301 MMDT2222A, Q302 DMP1045U-7, Q303 DMN313DLT-7, SW101 SW_Push, SW201 SW_Push, U201 STM32G431RBTx, U301 USBLC6-2SC6, U302 BQ25896RTW, U303 BQ27220YZFR, U305 BU33SD5WG-TR, U401 LSM6DSL, U402 DRV8833PW, U501 SN74AHCT1G125DBVR, Y201 X322516MLB4SI

Commit message: début du routing
Parts:
- moved C406 126.5 mm to (28.9, 115.5)
- moved U402 119.2 mm to (26.2, 124.8), turned to 0 degrees
- moved R404 117.4 mm to (32.8, 123.0), turned to 0 degrees
- moved R407 107.7 mm to (32.8, 125.9)
- moved R406 106.1 mm to (44.6, 118.4)
- moved C403 99.5 mm to (47.5, 114.4), turned to 0 degrees
- moved C405 98.1 mm to (47.5, 118.3), turned to 0 degrees
- moved R405 97.5 mm to (44.6, 116.4), turned to 0 degrees
- moved C404 97.2 mm to (47.5, 116.3), turned to 0 degrees
- moved J503 95.0 mm to (154.0, 55.0), turned to 180 degrees
- moved J301 93.4 mm to (138.9, 146.3), turned to 0 degrees
- moved J501 88.4 mm to (132.0, 55.0), turned to 180 degrees
- moved J506 87.2 mm to (122.0, 143.0), turned to 0 degrees
- moved J509 16.7 mm to (176.5, 55.0)
- moved C210 16.2 mm to (139.2, 94.9), turned to 180 degrees
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Connections:
- U402 pad 10: /STM32/TIM2_PWM_DRIVER3 -> /STM32/TIM2_PWM_DRIVER4
- U402 pad 2: /Connectors/2_Motor_+ -> /Connectors/1_Motor_+
- U402 pad 4: /Connectors/2_Motor_- -> /Connectors/1_Motor_-
- U402 pad 5: /Connectors/1_Motor_+ -> /Connectors/2_Motor_-
- U402 pad 7: /Connectors/1_Motor_- -> /Connectors/2_Motor_+
- U402 pad 9: /STM32/TIM2_PWM_DRIVER4 -> /STM32/TIM2_PWM_DRIVER3
Routing:
- net /Connectors/1_Encoder_B: track 53.1 -> 0.00 mm
- net /Connectors/1_Encoder_A: track 52.9 -> 0.00 mm
- net /STM32/TIM2_PWM_DRIVER1: track 29.6 -> 0.00 mm, vias 2 -> 0
- net /STM32/TIM2_PWM_DRIVER2: track 28.4 -> 0.00 mm, vias 2 -> 0
- net /STM32/TIM2_PWM_DRIVER4: track 23.9 -> 0.00 mm
- net /STM32/TIM2_PWM_DRIVER3: track 21.5 -> 0.00 mm
- net +5V: track 13.6 -> 0.00 mm, vias 2 -> 0
- net +3.3V: track 30.7 -> 24.3 mm, vias 8 -> 0
- net Net-(U402-AISEN): track 4.65 -> 0.00 mm
- net Net-(U402-BISEN): track 4.49 -> 0.00 mm
- net Net-(U402-VCP): track 2.27 -> 0.00 mm
- net Net-(U402-VINT): track 2.25 -> 0.00 mm
- net Net-(U402-~{SLEEP}): track 1.97 -> 0.00 mm
- net /STM32/FAULT: track 1.60 -> 0.00 mm
- net /STM32/SYS_SWDIO: track 34.6 -> 33.1 mm
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- removed copper zone on In1.Cu, net +3.3V
- removed copper zone on F.Cu, net /Connectors/1_Motor_+
- removed copper zone on F.Cu, net /Connectors/1_Motor_-
- removed copper zone on F.Cu, net /Connectors/2_Motor_+
- removed copper zone on F.Cu, net /Connectors/2_Motor_-
