File: Hardware/1ST_Schematix/_restore_backup_2026-10-05T08-37-58-085/Sensors&Driver_Inhibot.kicad_sch (KiCad schematic)
At the start: 19 parts, among them J511_OUT401 Conn_01x06, U401 LSM6DSL, U402 DRV8833PW

Commit message: début du routing
Connections:
- net AOUT1: now also U402.2 (AOUT1); no longer U402.5 (BOUT2)
- net AOUT2: now also U402.4 (AOUT2); no longer U402.7 (BOUT1)
- net BOUT1: now also U402.7 (BOUT1); no longer U402.2 (AOUT1)
- net BOUT2: now also U402.5 (BOUT2); no longer U402.4 (AOUT2)
- net PWM3: now also U402.9 (BIN1); no longer U402.10 (BIN2)
- net PWM4: now also U402.10 (BIN2); no longer U402.9 (BIN1)
Changed lines of the file:
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@@
 	(hierarchical_label "PWM4"
 		(shape input)
-		(at 195.58 106.68 180)
+		(at 195.58 109.22 180)
 		(effects
 			(font
@@
 	(hierarchical_label "AOUT2"
 		(shape output)
-		(at 220.98 106.68 0)
+		(at 220.98 104.14 0)
 		(effects
 			(font
@@
 	(hierarchical_label "PWM3"
 		(shape input)
-		(at 195.58 109.22 180)
+		(at 195.58 106.68 180)
 		(effects
 			(font
@@
 	(hierarchical_label "BOUT1"
 		(shape output)
-		(at 220.98 101.6 0)
+		(at 220.98 106.68 0)
 		(effects
 			(font
@@
 	(hierarchical_label "BOUT2"
 		(shape output)
-		(at 220.98 104.14 0)
+		(at 220.98 109.22 0)
 		(effects
 			(font
@@
 	(hierarchical_label "AOUT1"
 		(shape output)
-		(at 220.98 109.22 0)
+		(at 220.98 101.6 0)
 		(effects
 			(font
