File: Hardware/1ST_Schematix/_restore_backup_2026-10-07T08-19-37-846/1ST_Schematix.kicad_sch (KiCad schematic)
At the start: 6 parts, among them SW101 SW_Push

Commit message: fin du routage, plus qu'à faire le jlcpb
Parts:
- R101: JLCPCB Parts # r -> (none); now in the parts list
- SW101: JLCPCB Parts # C9900091799r -> (none)
Changed lines of the file:
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@@
-			)
-		)
-		(property "JLCPCB Parts #" "C9900091799\r"
-			(at 85.09 83.82 90)
-			(hide yes)
-			(show_name no)
-			(do_not_autoplace no)
-			(effects
-				(font
-					(size 1.27 1.27)
-				)
 			)
 		)
@@
 		(body_style 1)
 		(exclude_from_sim no)
-		(in_bom no)
+		(in_bom yes)
 		(on_board yes)
 		(in_pos_files yes)
@@
 			(at 85.09 69.85 0)
 			(hide yes)
-			(show_name no)
-			(do_not_autoplace no)
-			(effects
-				(font
-					(size 1.27 1.27)
-				)
-			)
-		)
-		(property "JLCPCB Parts #" "\r"
-			(at 85.09 69.85 0)
-			(hide yes)
