File: Hardware/1ST_Schematix/_restore_backup_2026-10-07T08-19-37-846/CPU_Inhibot.kicad_sch (KiCad schematic)
At the start: 22 parts, among them J201 Conn_ST_STDC14, SW201 SW_Push, U201 STM32G431RBT6, Y201 X322516MLB4SI

Commit message: fin du routage, plus qu'à faire le jlcpb
Parts:
- C201, C204, C205, C206, C209, C210: JLCPCB Part # (none) -> C1525; JLCPCB Parts # C1525 -> (none)
- C202, C203: JLCPCB Parts # C32949 -> (none)
- C207: JLCPCB Parts # C15195 -> (none)
- C208: JLCPCB Parts # C23733 -> (none)
- D201: JLCPCB Parts # C12624 -> (none)
- D202: JLCPCB Parts # C2286 -> (none)
- J201: JLCPCB Parts # C3975190 -> (none)
- R202, R203: JLCPCB Parts # C11702r -> (none)
- R205, R206: JLCPCB Parts # r -> (none); now in the parts list
- R207, R208: JLCPCB Parts # C25900r -> (none)
- SW201: JLCPCB Parts # C9900091799r -> (none)
- U201: value STM32G431RBT6 -> STM32G431RBTx; JLCPCB Parts # C431633r -> (none)
- Y201: JLCPCB Part # (none) -> C13738; JLCPCB Parts # C13738 -> (none)
Changed lines of the file:
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@@
 			)
 		)
-		(property "JLCPCB Parts #" "C11702\r"
-			(at 55.88 180.34 0)
-			(hide yes)
-			(show_name no)
-			(do_not_autoplace no)
-			(effects
-				(font
-					(size 1.27 1.27)
-				)
-			)
-		)
 		(pin "2"
 		)
@@
 			)
 		)
-		(property "KLC_S3.3" ""
+		(property "JLCPCB Part #" "C1525"
 			(at 69.85 31.75 0)
 			(hide yes)
@@
 			)
 		)
-		(property "KLC_S4.1" ""
+		(property "KLC_S3.3" ""
 			(at 69.85 31.75 0)
 			(hide yes)
@@
 			)
 		)
-		(property "JLCPCB Parts #" "C1525"
+		(property "KLC_S4.1" ""
 			(at 69.85 31.75 0)
 			(hide yes)
@@
 			)
 		)
-		(property "KLC_S3.3" ""
+		(property "JLCPCB Part #" "C1525"
 			(at 46.99 31.75 0)
 			(hide yes)
@@
 			)
 		)
-		(property "KLC_S4.1" ""
+		(property "KLC_S3.3" ""
 			(at 46.99 31.75 0)
 			(hide yes)
@@
 			)
 		)
-		(property "JLCPCB Parts #" "C1525"
+		(property "KLC_S4.1" ""
 			(at 46.99 31.75 0)
 			(hide yes)
@@
 			)
 		)
-		(property "JLCPCB Parts #" "C32949"
-			(at 34.29 63.5 90)
-			(hide yes)
-			(show_name no)
-			(do_not_autoplace no)
-			(effects
-				(font
-					(size 1.27 1.27)
-				)
-			)
-		)
 		(pin "1"
 		)
@@
 			)
 		)
-		(property "JLCPCB Parts #" "C23733"
-			(at 25.4 31.75 0)
-			(hide yes)
-			(show_name no)
-			(do_not_autoplace no)
-			(effects
-				(font
-					(size 1.27 1.27)
-				)
-			)
-		)
 		(pin "1"
 		)
@@
 			)
 		)
-		(property "JLCPCB Parts #" "C3975190"
-			(at 245.11 46.99 0)
-			(hide yes)
-			(show_name no)
-			(do_not_autoplace no)
-			(effects
-				(font
-					(size 1.27 1.27)
-				)
-			)
-		)
 		(pin "4"
 		)
@@
 			)
 		)
-		(property "Value" "STM32G431RBT6"
+		(property "Value" "STM32G431RBTx"
 			(at 101.2033 135.89 0)
 			(show_name no)
@@
 			)
 		)
-		(property "JLCPCB Parts #" "C431633\r"
-			(at 96.52 85.09 0)
-			(hide yes)
-			(show_name no)
-			(do_not_autoplace no)
-			(effects
-				(font
-					(size 1.27 1.27)
-				)
-			)
-		)
 		(pin "8"
 		)
@@
 			)
 		)
-		(property "JLCPCB Parts #" "C2286"
-			(at 76.2 173.99 90)
-			(hide yes)
-			(show_name no)
-			(do_not_autoplace no)
-			(effects
-				(font
-					(size 1.27 1.27)
-				)
-			)
-		)
 		(pin "2"
 		)
@@
 			)
 		)
-		(property "JLCPCB Parts #" "C9900091799\r"
-			(at 29.21 179.07 90)
-			(hide yes)
-			(show_name no)
-			(do_not_autoplace no)
-			(effects
-				(font
-					(size 1.27 1.27)
-				)
-			)
-		)
 		(pin "1"
 		)
@@
 		(body_style 1)
 		(exclude_from_sim no)
-		(in_bom no)
+		(in_bom yes)
 		(on_board yes)
 		(in_pos_files yes)
@@
 			)
 		)
-		(property "JLCPCB Parts #" "\r"
-			(at 180.34 93.98 0)
-			(hide yes)
-			(show_name no)
-			(do_not_autoplace no)
-			(effects
-				(font
-					(size 1.27 1.27)
-				)
-			)
-		)
 		(pin "2"
 		)
@@
 			)
 		)
-		(property "KLC_S3.3" ""
+		(property "JLCPCB Part #" "C1525"
 			(at 24.13 179.07 0)
 			(hide yes)
@@
 			)
 		)
-		(property "KLC_S4.1" ""
+		(property "KLC_S3.3" ""
 			(at 24.13 179.07 0)
 			(hide yes)
@@
 			)
 		)
-		(property "JLCPCB Parts #" "C1525"
+		(property "KLC_S4.1" ""
 			(at 24.13 179.07 0)
 			(hide yes)
@@
 			)
 		)
-		(property "JLCPCB Parts #" "C12624"
-			(at 55.88 172.72 90)
-			(hide yes)
-			(show_name no)
-			(do_not_autoplace no)
-			(effects
-				(font
-					(size 1.27 1.27)
-				)
-			)
-		)
 		(pin "2"
 		)
@@
 			)
 		)
-		(property "JLCPCB Parts #" "C13738"
+		(property "JLCPCB Part #" "C13738"
 			(at 43.18 58.42 90)
 			(hide yes)
@@
 			)
 		)
-		(property "JLCPCB Parts #" "C25900\r"
-			(at 191.77 121.92 0)
-			(hide yes)
-			(show_name no)
-			(do_not_autoplace no)
-			(effects
-				(font
-					(size 1.27 1.27)
-				)
-			)
-		)
 		(pin "2"
 		)
@@
 			)
 		)
-		(property "KLC_S3.3" ""
+		(property "JLCPCB Part #" "C1525"
 			(at 58.42 31.75 0)
 			(hide yes)
@@
 			)
 		)
-		(property "KLC_S4.1" ""
+		(property "KLC_S3.3" ""
 			(at 58.42 31.75 0)
 			(hide yes)
@@
 			)
 		)
-		(property "JLCPCB Parts #" "C1525"
+		(property "KLC_S4.1" ""
 			(at 58.42 31.75 0)
 			(hide yes)
@@
 			)
 		)
-		(property "JLCPCB Parts #" "C11702\r"
-			(at 76.2 181.61 0)
-			(hide yes)
-			(show_name no)
-			(do_not_autoplace no)
-			(effects
-				(font
-					(size 1.27 1.27)
-				)
-			)
-		)
 		(pin "2"
 		)
@@
 			)
 		)
-		(property "JLCPCB Parts #" "C25900\r"
-			(at 180.34 121.92 0)
-			(hide yes)
-			(show_name no)
-			(do_not_autoplace no)
-			(effects
-				(font
-					(size 1.27 1.27)
-				)
-			)
-		)
 		(pin "2"
 		)
@@
 			)
 		)
-		(property "KLC_S3.3" ""
+		(property "JLCPCB Part #" "C1525"
 			(at 35.56 31.75 0)
 			(hide yes)
@@
 			)
 		)
-		(property "KLC_S4.1" ""
+		(property "KLC_S3.3" ""
 			(at 35.56 31.75 0)
 			(hide yes)
@@
 			)
 		)
-		(property "JLCPCB Parts #" "C1525"
+		(property "KLC_S4.1" ""
 			(at 35.56 31.75 0)
 			(hide yes)
@@
 		(body_style 1)
 		(exclude_from_sim no)
-		(in_bom no)
+		(in_bom yes)
 		(on_board yes)
 		(in_pos_files yes)
@@
 			)
 		)
-		(property "JLCPCB Parts #" "\r"
-			(at 191.77 93.98 0)
-			(hide yes)
-			(show_name no)
-			(do_not_autoplace no)
-			(effects
-				(font
-					(size 1.27 1.27)
-				)
-			)
-		)
 		(pin "2"
 		)
@@
 			)
 		)
-		(property "KLC_S3.3" ""
+		(property "JLCPCB Part #" "C1525"
 			(at 69.85 39.37 0)
 			(hide yes)
@@
 			)
 		)
-		(property "KLC_S4.1" ""
+		(property "KLC_S3.3" ""
 			(at 69.85 39.37 0)
 			(hide yes)
@@
 			)
 		)
-		(property "JLCPCB Parts #" "C1525"
+		(property "KLC_S4.1" ""
 			(at 69.85 39.37 0)
 			(hide yes)
@@
 			)
 		)
-		(property "JLCPCB Parts #" "C32949"
-			(at 34.29 54.61 90)
-			(hide yes)
-			(show_name no)
-			(do_not_autoplace no)
-			(effects
-				(font
-					(size 1.27 1.27)
-				)
-			)
-		)
 		(pin "1"
 		)
@@
 			(at 119.38 33.02 0)
 			(hide yes)
-			(show_name no)
-			(do_not_autoplace no)
-			(effects
-				(font
-					(size 1.27 1.27)
-				)
-			)
-		)
-		(property "JLCPCB Parts #" "C15195"
-			(at 119.38 33.02 0)
-			(hide yes)
