File: Hardware/1ST_Schematix/_restore_backup_2026-10-07T08-19-37-846/Connector_Inhibot.kicad_sch (KiCad schematic)
At the start: 22 parts, among them J501 Conn_01x06, J502 Conn_01x03, J503 Conn_01x06, J504 Conn_01x05, J506 Conn_01x03, J507 Conn_01x03, J508 Conn_01x06, J509 Conn_01x06, J510 Conn_01x06, J511 Conn_01x03, U501 SN74AHCT1G125DBVR

Commit message: fin du routage, plus qu'à faire le jlcpb
Parts:
- removed C501, C504: 1u, Capacitor_SMD:C_0402_1005Metric, symbol Device:C_Small
- removed C505, C506, C507, C508, C509, C510: 100n, Capacitor_SMD:C_0402_1005Metric, symbol Device:C_Small
- C502, C503: JLCPCB Part # (none) -> C1525; JLCPCB Parts # C1525 -> (none)
- D502: JLCPCB Part # (none) -> C527089; JLCPCB Parts # C527089 -> (none)
- U501: JLCPCB Part # (none) -> C20617903; JLCPCB Parts # C20617903 -> (none)
