File: Hardware/1ST_Schematix/_restore_backup_2026-10-07T08-19-37-846/Power_Inhibot.kicad_sch (KiCad schematic)
At the start: 50 parts, among them J301 USB_C_Receptacle_USB2.0_16P, J302 Conn_01x02, Q301 MMDT2222A, Q302 DMP1045U-7, Q303 DMN313DLT-7, U301 USBLC6-2SC6, U302 BQ25896RTWR, U303 BQ27220YZFR, U305 BU33SD5WG-TR

Commit message: fin du routage, plus qu'à faire le jlcpb
Parts:
- C301: JLCPCB Part # (none) -> C1525; JLCPCB Parts # C1525 -> (none)
- C302: JLCPCB Parts # C1623 -> (none)
- C303: JLCPCB Parts # C12530 -> (none)
- C304: JLCPCB Parts # C880605 -> (none)
- C305: JLCPCB Parts # C23733 -> (none)
- C306, C307, C308, C309: JLCPCB Parts # C15525 -> (none)
- C310: JLCPCB Parts # C2182568 -> (none)
- C311, C312, C314: JLCPCB Parts # C52923 -> (none)
- D302: JLCPCB Parts # C12624 -> (none)
- D303: JLCPCB Parts # C111340 -> (none)
- J302: now in the parts list
- L301: footprint Inductor_SMD:L_0402_1005Metric -> Package_SO:SOIC-16_3.9x9.9mm_P1.27mm; JLCPCB Part # (none) -> MPL1608S1R0MHT; JLCPCB Parts # C84468r -> (none)
- Q301: JLCPCB Parts # C7603394r -> (none)
- Q302: JLCPCB Parts # C177033r -> (none)
- Q303: JLCPCB Parts # C155524r -> (none)
- R301, R304: JLCPCB Parts # C25741r -> (none)
- R302, R303, R312, R313: JLCPCB Parts # C25905r -> C25905
- R305: JLCPCB Parts # C11702r -> (none)
- R306: JLCPCB Part # (none) -> C105142; JLCPCB Parts # C105142r -> (none)
- R307, R309, R310, R311, R315, R316: JLCPCB Parts # C25744r -> (none)
- R308: JLCPCB Parts # C25117r -> (none)
- R314: JLCPCB Parts # C25076r -> (none)
- R317: value 4.7k -> 4k7; JLCPCB Parts # C25900r -> (none)
- U301: JLCPCB Parts # C7519r -> C7519
- U302: value BQ25896RTWR -> BQ25896RTW; JLCPCB Parts # C181475r -> (none)
- U303: JLCPCB Parts # C528617r -> (none)
- U305: JLCPCB Parts # C3750265r -> (none)
