File: Hardware/1ST_Schematix/_restore_backup_2026-10-07T08-19-37-846/Sensors&Driver_Inhibot.kicad_sch (KiCad schematic)
At the start: 19 parts, among them J511_OUT401 Conn_01x06, U401 LSM6DSL, U402 DRV8833PW-PR

Commit message: fin du routage, plus qu'à faire le jlcpb
Parts:
- C401, C402: JLCPCB Part # (none) -> C1525; JLCPCB Parts # C1525 -> (none)
- C403: JLCPCB Parts # C15195 -> (none)
- C404: JLCPCB Parts # C12530 -> (none)
- C405: JLCPCB Parts # C15525 -> (none)
- C406: JLCPCB Part # (none) -> C178566; JLCPCB Parts # C178566 -> (none)
- R401, R402, R403, R405, R406: JLCPCB Parts # C11702r -> (none)
- R404, R407: JLCPCB Part # (none) -> C2074761; JLCPCB Parts # C2074761r -> (none)
- R408: JLCPCB Parts # C25744r -> (none)
- U401: JLCPCB Parts (none) -> C126672; JLCPCB Parts # C126672r -> (none)
- U402: value DRV8833PW-PR -> DRV8833PW; footprint Package_SO:TSSOP-16-1EP_4.4x5mm_P0.65mm_EP3x3mm -> Package_SO:TSSOP-16_4.4x5mm_P0.65mm; JLCPCB Parts # C50506r -> (none)
Changed lines of the file:
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@@
 			)
 		)
-		(property "JLCPCB Parts #" "C11702\r"
-			(at 63.5 92.71 90)
-			(hide yes)
-			(show_name no)
-			(do_not_autoplace no)
-			(effects
-				(font
-					(size 1.27 1.27)
-				)
-			)
-		)
 		(pin "2"
 		)
@@
 			)
 		)
-		(property "JLCPCB Parts #" "C12530"
-			(at 208.28 73.66 90)
-			(hide yes)
-			(show_name no)
-			(do_not_autoplace no)
-			(effects
-				(font
-					(size 1.27 1.27)
-				)
-			)
-		)
 		(pin "2"
 		)
@@
 			)
 		)
-		(property "JLCPCB Parts #" "C11702\r"
-			(at 71.12 102.87 90)
-			(hide yes)
-			(show_name no)
-			(do_not_autoplace no)
-			(effects
-				(font
-					(size 1.27 1.27)
-				)
-			)
-		)
 		(pin "2"
 		)
@@
 			)
 		)
-		(property "JLCPCB Parts #" "C25744\r"
-			(at 63.5 86.36 90)
-			(hide yes)
-			(show_name no)
-			(do_not_autoplace no)
-			(effects
-				(font
-					(size 1.27 1.27)
-				)
-			)
-		)
 		(pin "2"
 		)
@@
 			)
 		)
-		(property "KLC_S3.3" ""
+		(property "JLCPCB Part #" "C2074761"
 			(at 177.8 97.79 90)
 			(hide yes)
@@
 			)
 		)
-		(property "KLC_S4.1" ""
+		(property "KLC_S3.3" ""
 			(at 177.8 97.79 90)
 			(hide yes)
@@
 			)
 		)
-		(property "JLCPCB Parts #" "C2074761\r"
+		(property "KLC_S4.1" ""
 			(at 177.8 97.79 90)
 			(hide yes)
@@
 			)
 		)
-		(property "KLC_S3.3" ""
+		(property "JLCPCB Parts" "C126672"
 			(at 88.9 95.25 0)
 			(hide yes)
@@
 			)
 		)
-		(property "KLC_S4.1" ""
+		(property "KLC_S3.3" ""
 			(at 88.9 95.25 0)
 			(hide yes)
@@
 			)
 		)
-		(property "JLCPCB Parts #" "C126672\r"
+		(property "KLC_S4.1" ""
 			(at 88.9 95.25 0)
 			(hide yes)
@@
 			)
 		)
-		(property "JLCPCB Parts #" "C11702\r"
-			(at 237.49 93.98 90)
-			(hide yes)
-			(show_name no)
-			(do_not_autoplace no)
-			(effects
-				(font
-					(size 1.27 1.27)
-				)
-			)
-		)
 		(pin "1"
 		)
@@
 			)
 		)
-		(property "JLCPCB Parts #" "C15525"
-			(at 223.52 80.01 90)
-			(hide yes)
-			(show_name no)
-			(do_not_autoplace no)
-			(effects
-				(font
-					(size 1.27 1.27)
-				)
-			)
-		)
 		(pin "2"
 		)
@@
 			)
 		)
-		(property "JLCPCB Parts #" "C11702\r"
-			(at 63.5 90.17 90)
-			(hide yes)
-			(show_name no)
-			(do_not_autoplace no)
-			(effects
-				(font
-					(size 1.27 1.27)
-				)
-			)
-		)
 		(pin "2"
 		)
@@
 			)
 		)
-		(property "JLCPCB Parts #" "C15195"
-			(at 185.42 82.55 0)
-			(hide yes)
-			(show_name no)
-			(do_not_autoplace no)
-			(effects
-				(font
-					(size 1.27 1.27)
-				)
-			)
-		)
 		(pin "1"
 		)
@@
 			)
 		)
-		(property "JLCPCB Parts #" ""
-			(at 50.8 128.27 0)
-			(hide yes)
-			(show_name no)
-			(do_not_autoplace no)
-			(effects
-				(font
-					(size 1.27 1.27)
-				)
-			)
-		)
 		(pin "1"
 		)
@@
 			)
 		)
-		(property "KLC_S3.3" ""
+		(property "JLCPCB Part #" "C178566"
 			(at 236.22 80.01 0)
 			(hide yes)
@@
 			)
 		)
-		(property "KLC_S4.1" ""
+		(property "KLC_S3.3" ""
 			(at 236.22 80.01 0)
 			(hide yes)
@@
 			)
 		)
-		(property "JLCPCB Parts #" "C178566"
+		(property "KLC_S4.1" ""
 			(at 236.22 80.01 0)
 			(hide yes)
@@
 			)
 		)
-		(property "Value" "DRV8833PW-PR"
+		(property "Value" "DRV8833PW"
 			(at 210.4233 116.84 0)
 			(show_name no)
@@
 			)
 		)
-		(property "Footprint" "Package_SO:TSSOP-16-1EP_4.4x5mm_P0.65mm_EP3x3mm"
+		(property "Footprint" "Package_SO:TSSOP-16_4.4x5mm_P0.65mm"
 			(at 213.36 116.84 0)
 			(hide yes)
@@
 			)
 		)
-		(property "JLCPCB Parts #" "C50506\r"
-			(at 208.28 99.06 0)
-			(hide yes)
-			(show_name no)
-			(do_not_autoplace no)
-			(effects
-				(font
-					(size 1.27 1.27)
-				)
-			)
-		)
 		(pin "16"
 		)
@@
 			)
 		)
-		(property "JLCPCB Parts #" "C11702\r"
-			(at 195.58 81.28 90)
-			(hide yes)
-			(show_name no)
-			(do_not_autoplace no)
-			(effects
-				(font
-					(size 1.27 1.27)
-				)
-			)
-		)
 		(pin "1"
 		)
@@
 			)
 		)
-		(property "KLC_S3.3" ""
+		(property "JLCPCB Part #" "C1525"
 			(at 95.25 74.93 0)
 			(hide yes)
@@
 			)
 		)
-		(property "KLC_S4.1" ""
+		(property "KLC_S3.3" ""
 			(at 95.25 74.93 0)
 			(hide yes)
@@
 			)
 		)
-		(property "JLCPCB Parts #" "C1525"
+		(property "KLC_S4.1" ""
 			(at 95.25 74.93 0)
 			(hide yes)
@@
 			)
 		)
-		(property "KLC_S3.3" ""
+		(property "JLCPCB Part #" "C2074761"
 			(at 177.8 105.41 90)
 			(hide yes)
@@
 			)
 		)
-		(property "KLC_S4.1" ""
+		(property "KLC_S3.3" ""
 			(at 177.8 105.41 90)
 			(hide yes)
@@
 			)
 		)
-		(property "JLCPCB Parts #" "C2074761\r"
+		(property "KLC_S4.1" ""
 			(at 177.8 105.41 90)
 			(hide yes)
@@
 			)
 		)
-		(property "KLC_S3.3" ""
+		(property "JLCPCB Part #" "C1525"
 			(at 85.09 74.93 0)
 			(hide yes)
@@
 			)
 		)
-		(property "KLC_S4.1" ""
+		(property "KLC_S3.3" ""
 			(at 85.09 74.93 0)
 			(hide yes)
@@
 			)
 		)
-		(property "JLCPCB Parts #" "C1525"
+		(property "KLC_S4.1" ""
 			(at 85.09 74.93 0)
 			(hide yes)
