File: Hardware/1ST_Schematix/_restore_backup_2026-10-07T10-14-57-809/Connector_Inhibot.kicad_sch (KiCad schematic)
At the start: 22 parts, among them J501 Conn_01x06, J502 Conn_01x03, J503 Conn_01x06, J504 Conn_01x05, J506 Conn_01x03, J507 Conn_01x03, J508 Conn_01x06, J509 Conn_01x06, J510 Conn_01x06, J511 Conn_01x03, U501 SN74AHCT1G125DBVR

Commit message: fin du routage, plus qu'à faire le jlcpb
Parts:
- C501, C504: JLCPCB Parts # C52923 -> (none)
- C502, C503, C505, C506, C507, C508, C509, C510: JLCPCB Part # (none) -> C1525; JLCPCB Parts # C1525 -> (none)
- D502: JLCPCB Part # (none) -> C527089; JLCPCB Parts # C527089 -> (none)
- U501: JLCPCB Part # (none) -> C20617903; JLCPCB Parts # C20617903 -> (none)
Changed lines of the file:
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@@
 			)
 		)
-		(property "JLCPCB Parts #" ""
-			(at 60.96 43.18 0)
-			(hide yes)
-			(show_name no)
-			(do_not_autoplace no)
-			(effects
-				(font
-					(size 1.27 1.27)
-				)
-			)
-		)
 		(pin "1"
 		)
@@
 			)
 		)
-		(property "JLCPCB Parts #" ""
-			(at 45.72 43.18 0)
-			(hide yes)
-			(show_name no)
-			(do_not_autoplace no)
-			(effects
-				(font
-					(size 1.27 1.27)
-				)
-			)
-		)
 		(pin "1"
 		)
@@
 			)
 		)
-		(property "JLCPCB Parts #" ""
-			(at 233.68 97.79 0)
-			(hide yes)
-			(show_name no)
-			(do_not_autoplace no)
-			(effects
-				(font
-					(size 1.27 1.27)
-				)
-			)
-		)
 		(pin "1"
 		)
@@
 			)
 		)
-		(property "KLC_S3.3" ""
+		(property "JLCPCB Part #" "C527089"
 			(at 158.75 52.07 0)
 			(hide yes)
@@
 			)
 		)
-		(property "KLC_S4.1" ""
+		(property "KLC_S3.3" ""
 			(at 158.75 52.07 0)
 			(hide yes)
@@
 			)
 		)
-		(property "JLCPCB Parts #" "C527089"
+		(property "KLC_S4.1" ""
 			(at 158.75 52.07 0)
 			(hide yes)
@@
 			)
 		)
-		(property "KLC_S3.3" ""
+		(property "JLCPCB Part #" "C1525"
 			(at 25.4 43.18 0)
 			(hide yes)
@@
 			)
 		)
-		(property "KLC_S4.1" ""
+		(property "KLC_S3.3" ""
 			(at 25.4 43.18 0)
 			(hide yes)
@@
 			)
 		)
-		(property "JLCPCB Parts #" "C1525"
+		(property "KLC_S4.1" ""
 			(at 25.4 43.18 0)
 			(hide yes)
@@
 			)
 		)
-		(property "JLCPCB Parts #" ""
-			(at 231.14 55.88 0)
-			(hide yes)
-			(show_name no)
-			(do_not_autoplace no)
-			(effects
-				(font
-					(size 1.27 1.27)
-				)
-			)
-		)
 		(pin "1"
 		)
@@
 			)
 		)
-		(property "KLC_S3.3" ""
+		(property "JLCPCB Part #" "C1525"
 			(at 104.14 43.18 0)
 			(hide yes)
@@
 			)
 		)
-		(property "KLC_S4.1" ""
+		(property "KLC_S3.3" ""
 			(at 104.14 43.18 0)
 			(hide yes)
@@
 			)
 		)
-		(property "JLCPCB Parts #" "C1525"
+		(property "KLC_S4.1" ""
 			(at 104.14 43.18 0)
 			(hide yes)
@@
 			)
 		)
-		(property "KLC_S3.3" ""
+		(property "JLCPCB Part #" "C1525"
 			(at 82.55 43.18 0)
 			(hide yes)
@@
 			)
 		)
-		(property "KLC_S4.1" ""
+		(property "KLC_S3.3" ""
 			(at 82.55 43.18 0)
 			(hide yes)
@@
 			)
 		)
-		(property "JLCPCB Parts #" "C1525"
+		(property "KLC_S4.1" ""
 			(at 82.55 43.18 0)
 			(hide yes)
@@
 			)
 		)
-		(property "KLC_S3.3" ""
+		(property "JLCPCB Part #" "C20617903"
 			(at 119.38 52.07 0)
 			(hide yes)
@@
 			)
 		)
-		(property "KLC_S4.1" ""
+		(property "KLC_S3.3" ""
 			(at 119.38 52.07 0)
 			(hide yes)
@@
 			)
 		)
-		(property "JLCPCB Parts #" "C20617903"
+		(property "KLC_S4.1" ""
 			(at 119.38 52.07 0)
 			(hide yes)
@@
 			)
 		)
-		(property "JLCPCB Parts #" ""
-			(at 217.17 97.79 0)
-			(hide yes)
-			(show_name no)
-			(do_not_autoplace no)
-			(effects
-				(font
-					(size 1.27 1.27)
-				)
-			)
-		)
 		(pin "1"
 		)
@@
 			)
 		)
-		(property "JLCPCB Parts #" "C52923"
-			(at 153.67 96.52 0)
-			(hide yes)
-			(show_name no)
-			(do_not_autoplace no)
-			(effects
-				(font
-					(size 1.27 1.27)
-				)
-			)
-		)
 		(pin "2"
 		)
@@
 			)
 		)
-		(property "KLC_S3.3" ""
+		(property "JLCPCB Part #" "C1525"
 			(at 146.05 39.37 0)
 			(hide yes)
@@
 			)
 		)
-		(property "KLC_S4.1" ""
+		(property "KLC_S3.3" ""
 			(at 146.05 39.37 0)
 			(hide yes)
@@
 			)
 		)
-		(property "JLCPCB Parts #" "C1525"
+		(property "KLC_S4.1" ""
 			(at 146.05 39.37 0)
 			(hide yes)
@@
 			)
 		)
-		(property "KLC_S3.3" ""
+		(property "JLCPCB Part #" "C1525"
 			(at 71.12 129.54 0)
 			(hide yes)
@@
 			)
 		)
-		(property "KLC_S4.1" ""
+		(property "KLC_S3.3" ""
 			(at 71.12 129.54 0)
 			(hide yes)
@@
 			)
 		)
-		(property "JLCPCB Parts #" "C1525"
+		(property "KLC_S4.1" ""
 			(at 71.12 129.54 0)
 			(hide yes)
@@
 			)
 		)
-		(property "KLC_S3.3" ""
+		(property "JLCPCB Part #" "C1525"
 			(at 257.81 57.15 0)
 			(hide yes)
@@
 			)
 		)
-		(property "KLC_S4.1" ""
+		(property "KLC_S3.3" ""
 			(at 257.81 57.15 0)
 			(hide yes)
@@
 			)
 		)
-		(property "JLCPCB Parts #" "C1525"
+		(property "KLC_S4.1" ""
 			(at 257.81 57.15 0)
 			(hide yes)
@@
 			)
 		)
-		(property "JLCPCB Parts #" "C52923"
-			(at 127 97.79 0)
-			(hide yes)
-			(show_name no)
-			(do_not_autoplace no)
-			(effects
-				(font
-					(size 1.27 1.27)
-				)
-			)
-		)
 		(pin "2"
 		)
@@
 			)
 		)
-		(property "KLC_S3.3" ""
+		(property "JLCPCB Part #" "C1525"
 			(at 250.19 92.71 0)
 			(hide yes)
@@
 			)
 		)
-		(property "KLC_S4.1" ""
+		(property "KLC_S3.3" ""
 			(at 250.19 92.71 0)
 			(hide yes)
@@
 			)
 		)
-		(property "JLCPCB Parts #" "C1525"
+		(property "KLC_S4.1" ""
 			(at 250.19 92.71 0)
 			(hide yes)
@@
 			)
 		)
-		(property "KLC_S3.3" ""
+		(property "JLCPCB Part #" "C1525"
 			(at 199.39 92.71 0)
 			(hide yes)
@@
 			)
 		)
-		(property "KLC_S4.1" ""
+		(property "KLC_S3.3" ""
 			(at 199.39 92.71 0)
 			(hide yes)
@@
 			)
 		)
-		(property "JLCPCB Parts #" "C1525"
+		(property "KLC_S4.1" ""
 			(at 199.39 92.71 0)
 			(hide yes)
